File: pcb/FindMyCharger.kicad_sch (KiCad schematic)
At the start: 196 parts, among them IC1 CAV24C256WE-GT3, J1 USB_C_Receptacle, J2 USB_C_Receptacle, J3 Battery_Connector, Q1 Q_NMOS, Q2 Q_NMOS, Q3 Q_NMOS, Q4 Q_NMOS, Q5 Q_PMOS, Q6 Q_NMOS, Q7 Q_PMOS, Q8 Q_NMOS, Q9 Q_NMOS, SW1 SW_Push, SW2 SW_Push, SW3 SW_Push, U1 TPS25762CQRQLRQ1, U2 BQ25713BRSNT, U3 BQ4050RSMR, U5 nRF54L10-QFXX, U6 TPS25730DREFR, Y1 XTAL_2016

Commit message: update
Parts:
- H1, H10, H3, H4, H5, H6, H7, H8, H9: footprint (none) -> TestPoint:TestPoint_THTPad_D2.5mm_Drill1.2mm
- H2: footprint (none) -> TestPoint:TestPoint_THTPad_2.5x2.5mm_Drill1.2mm
Other:
- moved on the sheet: C43, D15, H7, R30, R35

Commit message: some esd
Parts:
- removed D2, D4, D5, D6: D_TVS, symbol Device:D_TVS
- added D19, D2, D21, D4, D5, D6: D_Zener, symbol Device:D_Zener
- added R66: 100, symbol Device:R
- R32, R34: value 470 -> 200
- R33: value 470 -> 100
- TH1: value Thermistor_NTC_47k -> 47k
Connections:
- net CC1_OUT: now also D4.1 (K)
- net CC2_OUT: now also D2.1 (K)
- net CHGND: now also C40.1, C52.2, C60.2, U3.9 (VSS); no longer R52.2
- net DM_OUT: now also D6.1 (K)
- net DP_OUT: now also D5.1 (K)
- net GND: now also R52.2, D19.2 (A), D2.2 (A), D21.2 (A), D4.2 (A), D5.2 (A), D6.2 (A); no longer C40.1, C42.2, R65.2, SW3.2, U3.14 (NC), U3.29 (NC), U3.9 (VSS)
- net at C48.1, J3.GND, R40.2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: no longer C52.2, C60.2
- net at H6.1: now also R33.2; no longer U3.18 (SMBD)
- net at H5.1: now also R66.2; no longer U3.19 (SMBC)
- net at U3.20 (LEDCNTLA): now also D1.2 (A), D3.1 (K), D9.1 (K); no longer R33.2
- net at U3.21 (LEDCNTLB): now also D1.1 (K), D3.2 (A), D7.2 (A), D8.1 (K); no longer R34.2
- net at U3.22 (LEDCNTLC): now also D7.1 (K), D8.2 (A), D9.2 (A); no longer R32.1
- new net: D19.1 (K), R32.2, R33.1
- new net: C42.2, R65.2, SW3.2
- new net: D21.1 (K), R34.2, R66.1
- new net BMS_SMBC: R34.1, U3.19 (SMBC)
- new net BMS_SMBD: R32.1, U3.18 (SMBD)
Other:
- moved on the sheet: C43, D1, D10, D11, D12, D13, D15, D16, D17, D18, D3, D7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

Commit message: more esd + research
Parts:
- removed D21: D_Zener, symbol Device:D_Zener
- removed J2: USB_C_Receptacle, Connector_USB:USB_C_Plug_Molex_105444, symbol Connector:USB_C_Receptacle
- added D20: D_Zener, symbol Device:D_Zener
- added J4: USB_C_Receptacle, symbol Connector:USB_C_Receptacle
Connections:
- net CC1_OUT: now also J4.A5 (CC1)
- net CC2_OUT: now also J4.B5 (CC2)
- net DM_OUT: now also J4.A7 (D-), J4.B7 (D-)
- net DP_OUT: now also J4.A6 (D+), J4.B6 (D+)
- net GND: now also D20.2 (A), J4.A1 (GND), J4.A12 (GND), J4.B1 (GND), J4.B12 (GND); no longer D10.2 (A2)
- net VBUS_OUT: now also J4.A4 (VBUS), J4.A9 (VBUS), J4.B4 (VBUS), J4.B9 (VBUS)
- net at H5.1, R66.2: now also D10.2 (A2)
- net at H6.1, R33.2: now also D11.2 (A2)
- net at R34.2, R66.1: now also D20.1 (K)
Other:
- moved on the sheet: H5, H6, R32, R33

Commit message: shield to gnd
Connections:
- net GND: now also J1.S1 (SHIELD), J4.SH (SHIELD)
- no-connect marks 12 -> 11
Changed lines of the file:
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@@
 	)
 	(junction
+		(at 24.13 110.49)
+		(diameter 0)
+		(color 0 0 0 0)
+	)
+	(junction
 		(at 654.05 109.22)
 		(diameter 0)
@@
 	)
 	(junction
+		(at 36.83 342.9)
+		(diameter 0)
+		(color 0 0 0 0)
+	)
+	(junction
 		(at 659.13 101.6)
 		(diameter 0)
@@
 	)
 	(no_connect
-		(at 33.02 342.9)
-	)
-	(no_connect
 		(at 55.88 320.04)
 	)
@@
 	(wire
 		(pts
+			(xy 20.32 110.49) (xy 24.13 110.49)
+		)
+		(stroke
+			(width 0)
+			(type default)
+		)
+	)
+	(wire
+		(pts
 			(xy 66.04 149.86) (xy 66.04 151.13)
 		)
@@
 	(wire
 		(pts
+			(xy 33.02 342.9) (xy 36.83 342.9)
+		)
+		(stroke
+			(width 0)
+			(type default)
+		)
+	)
+	(wire
+		(pts
 			(xy 175.26 347.98) (xy 175.26 349.25)
 		)
@@
 	(wire
 		(pts
+			(xy 36.83 342.9) (xy 40.64 342.9)
+		)
+		(stroke
+			(width 0)
+			(type default)
+		)
+	)
+	(wire
+		(pts
 			(xy 274.32 274.32) (xy 292.1 274.32)
 		)
@@
 	(wire
 		(pts
+			(xy 24.13 110.49) (xy 27.94 110.49)
+		)
+		(stroke
+			(width 0)
+			(type default)
+		)
+	)
+	(wire
+		(pts
 			(xy 46.99 373.38) (xy 46.99 372.11)
 		)
@@
 	(symbol
 		(lib_id "power:GND")
-		(at 40.64 342.9 0)
+		(at 36.83 342.9 0)
 		(unit 1)
 		(body_style 1)
@@
 		(fields_autoplaced yes)
 		(property "Reference" "#PWR03"
-			(at 40.64 349.25 0)
+			(at 36.83 349.25 0)
 			(hide yes)
 			(show_name no)
@@
 		)
 		(property "Value" "GND"
-			(at 40.64 347.98 0)
+			(at 36.83 347.98 0)
 			(show_name no)
 			(do_not_autoplace no)
@@
 		)
 		(property "Footprint" ""
-			(at 40.64 342.9 0)
+			(at 36.83 342.9 0)
 			(hide yes)
 			(show_name no)
@@
 		)
 		(property "Datasheet" ""
-			(at 40.64 342.9 0)
+			(at 36.83 342.9 0)
 			(hide yes)
 			(show_name no)
@@
 		)
 		(property "Description" "Power symbol creates a global label with name \"GND\" , ground"
-			(at 40.64 342.9 0)
+			(at 36.83 342.9 0)
 			(hide yes)
 			(show_name no)
@@
 	(symbol
 		(lib_id "power:GND")
-		(at 27.94 110.49 0)
+		(at 24.13 110.49 0)
 		(unit 1)
 		(body_style 1)
@@
 		(fields_autoplaced yes)
 		(property "Reference" "#PWR0101"
-			(at 27.94 116.84 0)
+			(at 24.13 116.84 0)
 			(hide yes)
 			(show_name no)
@@
 		)
 		(property "Value" "GND"
-			(at 27.94 115.57 0)
+			(at 24.13 115.57 0)
 			(show_name no)
 			(do_not_autoplace no)
@@
 		)
 		(property "Footprint" ""
-			(at 27.94 110.49 0)
+			(at 24.13 110.49 0)
 			(hide yes)
 			(show_name no)
@@
 		)
 		(property "Datasheet" ""
-			(at 27.94 110.49 0)
+			(at 24.13 110.49 0)
 			(hide yes)
 			(show_name no)
@@
 		)
 		(property "Description" "Power symbol creates a global label with name \"GND\" , ground"
-			(at 27.94 110.49 0)
+			(at 24.13 110.49 0)
 			(hide yes)
 			(show_name no)

Commit message: replace with non handsolder
Parts:
- added C55: 0.1uF, Capacitor_SMD:C_0603_1608Metric, symbol Device:C
- added H11: cSDA, TestPoint:TestPoint_THTPad_D2.5mm_Drill1.2mm, symbol Mechanical:MountingHole_Pad
- added H12: cSCL, TestPoint:TestPoint_THTPad_D2.5mm_Drill1.2mm, symbol Mechanical:MountingHole_Pad
- added R67, R68: 10k, symbol Device:R
- C1, C32, C40, C5, C50, C59: footprint Capacitor_SMD:C_0805_2012Metric_Pad1.18x1.45mm_HandSolder -> Capacitor_SMD:C_0805_2012Metric
- C10, C11, C13, C4, C6, C63, C65, C7, C71, C8: footprint Capacitor_SMD:C_1206_3216Metric_Pad1.33x1.80mm_HandSolder -> Capacitor_SMD:C_1206_3216Metric
- C12, C14, C15, C16, C17, C18, C19, C2, C20, C21, C22, C24, C25, C28, C3, C30, C33, C34, C35, C36, C37, C41, C42, C45, C46, C47, C48, C52, C56, C57, C58, C60, C61, C62, C64, C66, C68, C70, C72, C73, C9: footprint Capacitor_SMD:C_0603_1608Metric_Pad1.08x0.95mm_HandSolder -> Capacitor_SMD:C_0603_1608Metric
- C23, C67, C69: footprint Capacitor_SMD:C_1210_3225Metric_Pad1.33x2.70mm_HandSolder -> Capacitor_SMD:C_1210_3225Metric
- C26, C31: value 10V/0.1uF -> 0.1uF; footprint Capacitor_SMD:C_0603_1608Metric_Pad1.08x0.95mm_HandSolder -> Capacitor_SMD:C_0603_1608Metric; Power_Rating (none) -> 10V
- C27, C29, C39: footprint Capacitor_SMD:C_2225_5664Metric_Pad1.80x6.60mm_HandSolder -> Capacitor_SMD:C_2225_5664Metric
- C38: footprint Capacitor_SMD:C_1812_4532Metric_Pad1.57x3.40mm_HandSolder -> Capacitor_SMD:C_1812_4532Metric
- D9: footprint LED_SMD:LED_0603_1608Metric_Pad1.05x0.95mm_HandSolder -> LED_SMD:LED_0603_1608Metric
- H5: value SMBC -> bSMBC
- H6: value SMBD -> bSMBD
- R27, R28: Power_Rating 0.1W 50V -> 0.1W
- R30: Power_Rating (none) -> 0.1W
- R54: value 198.2k -> 198k
- R55: value 2.28k -> 2.20k
- R57: value 191k -> 198k
Connections:
- net GND: now also C55.2
- net OUTPUT_IN: now also C55.1
- net OUTPUT_LDO_3V3: now also R67.1, R68.1
- net CHG_SDA: now reaches U2.12 (SDA)
- net CHG_SDA: now also H11.1, R67.2
- net CHG_SCL: now reaches U2.13 (SCL)
- net CHG_SCL: now also H12.1, R68.2
Other:
- moved on the sheet: C22, C36, R19, R29, R9

Commit message: add 2010
Parts:
- R30: footprint (none) -> Resistor_SMD:R_2010_5025Metric
Changed lines of the file:
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@@
 			)
 		)
-		(property "Footprint" ""
+		(property "Footprint" "Resistor_SMD:R_2010_5025Metric"
 			(at 322.58 334.518 90)
 			(hide yes)

Commit message: fix SNS power rating
Parts:
- C1, C32, C40, C5, C50, C59: footprint Capacitor_SMD:C_0805_2012Metric -> Capacitor_SMD:C_0805_2012Metric_Pad1.18x1.45mm_HandSolder
- C10, C11, C13, C4, C6, C63, C65, C7, C71, C8: footprint Capacitor_SMD:C_1206_3216Metric -> Capacitor_SMD:C_1206_3216Metric_Pad1.33x1.80mm_HandSolder
- C12, C14, C15, C16, C17, C18, C19, C2, C20, C21, C22, C24, C25, C26, C28, C3, C30, C31, C33, C34, C35, C36, C37, C41, C42, C45, C46, C47, C48, C52, C55, C56, C57, C58, C60, C61, C62, C64, C66, C68, C70, C72, C73, C9: footprint Capacitor_SMD:C_0603_1608Metric -> Capacitor_SMD:C_0603_1608Metric_Pad1.08x0.95mm_HandSolder
- C23, C67, C69: footprint Capacitor_SMD:C_1210_3225Metric -> Capacitor_SMD:C_1210_3225Metric_Pad1.33x2.70mm_HandSolder
- C27, C29, C39: footprint Capacitor_SMD:C_2225_5664Metric -> Capacitor_SMD:C_2225_5664Metric_Pad1.80x6.60mm_HandSolder
- C38: footprint Capacitor_SMD:C_1812_4532Metric -> Capacitor_SMD:C_1812_4532Metric_Pad1.57x3.40mm_HandSolder
- D9: footprint LED_SMD:LED_0603_1608Metric -> LED_SMD:LED_0603_1608Metric_Pad1.05x0.95mm_HandSolder
- R30: Power_Rating 0.1W -> 0.33W

Commit message: some stuf
Parts:
- removed TH1: 47k, symbol Device:Thermistor_NTC
- added D21: D_Schottky, symbol Device:D_Schottky
- added R69: 6.65k, symbol Device:R
- added TH1: Thermistor, symbol Device:Thermistor
- C19, C20, C41, C42, C66, C68, C70: Power_Rating (none) -> 50V
- R17: Power_Rating (none) -> 0.5W
- R9: Power_Rating (none) -> 0.25W
Connections:
- net GND: now also C42.2, R65.2, SW3.2, D21.2 (A)
- net OUTPUT_LDO_3V3: now also TH1.1
- net OUTPUT_NTC: now also TH1.2
- net OUTPUT_TVSP: now also R69.1; no longer SW3.1
- net VBUS_IN: now also D21.1 (K)
- new net: R69.2, SW3.1
Other:
- note added: "20V max"
- note added: "3A max"
- note added: "3A min"
- note added: "5V min"
- moved on the sheet: C42, C63, C64, C66, C67, C68, C69, C70, C71, C72, C73, R60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
