File: pcb/FindMyCharger.kicad_sch (KiCad schematic)
At the start: 215 parts, among them IC1 CAV24C256WE-GT3, J1 USB_C_Receptacle, J3 Battery_Connector, J4 USB_C_Receptacle, Q1 Q_NMOS, Q2 Q_NMOS, Q3 Q_NMOS, Q4 Q_NMOS, Q5 Q_PMOS, Q6 Q_NMOS, Q7 Q_PMOS, Q8 Q_NMOS, Q9 Q_NMOS, SW1 SW_Push, SW2 SW_Push, SW3 SW_Push, U1 TPS25762CQRQLRQ1, U2 BQ25713RSNT, U3 BQ4050RSMR, U5 nRF54L10-QFXX, U6 TPS25730DREFR, Y1 32Mhz

Commit message: maaths
Parts:
- C42: Power_Rating 50V -> 40V
- J1, J4: footprint (none) -> Connector_USB:USB_C_Receptacle_GCT_USB4105-xx-A_16P_TopMnt_Horizontal
- R69: value 6.65k -> 5.6k; Tolerance (none) -> 1%
- U1: value TPS25762CQRQLRQ1 -> TPS25762DQRQLRQ1; LCSC Part (none) -> C43131301; MPN (none) -> TPS25762DQRQLRQ1
- U2: value BQ25713RSNT -> BQ25713RSNR; LCSC Part (none) -> C2878935; MPN (none) -> BQ25713RSNR
- U5: footprint Package_DFN_QFN:QFN-48-1EP_6x6mm_P0.4mm_EP4.6x4.6mm -> Package_DFN_QFN:QFN-48-1EP_6x6mm_P0.4mm_EP4.6x4.6mm_ThermalVias; LCSC Part (none) -> C44800139; MPN (none) -> NRF54L10-QFAA-R7
Changed lines of the file:
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@@
 			)
 		)
-		(property "Power_Rating" "50V"
+		(property "Power_Rating" "40V"
 			(at 55.88 387.35 0)
 			(hide yes)
@@
 			)
 		)
-		(property "Footprint" ""
+		(property "Footprint" "Connector_USB:USB_C_Receptacle_GCT_USB4105-xx-A_16P_TopMnt_Horizontal"
 			(at 41.91 302.26 0)
 			(hide yes)
@@
 			)
 		)
-		(property "Value" "TPS25762CQRQLRQ1"
+		(property "Value" "TPS25762DQRQLRQ1"
 			(at 132.08 293.37 0)
 			(show_name no)
@@
 			)
 		)
-		(property "MPN" ""
+		(property "MPN" "TPS25762DQRQLRQ1"
 			(at 88.9 300.99 0)
 			(hide yes)
@@
 			)
 		)
+		(property "Dielectric" ""
+			(at 88.9 300.99 0)
+			(hide yes)
+			(show_name no)
+			(do_not_autoplace no)
+			(effects
+				(font
+					(size 1.27 1.27)
+				)
+			)
+		)
+		(property "Tolerance" ""
+			(at 88.9 300.99 0)
+			(hide yes)
+			(show_name no)
+			(do_not_autoplace no)
+			(effects
+				(font
+					(size 1.27 1.27)
+				)
+			)
+		)
+		(property "Voltage" ""
+			(at 88.9 300.99 0)
+			(hide yes)
+			(show_name no)
+			(do_not_autoplace no)
+			(effects
+				(font
+					(size 1.27 1.27)
+				)
+			)
+		)
+		(property "Type" ""
+			(at 88.9 300.99 0)
+			(hide yes)
+			(show_name no)
+			(do_not_autoplace no)
+			(effects
+				(font
+					(size 1.27 1.27)
+				)
+			)
+		)
+		(property "LCSC Part" "C43131301"
+			(at 88.9 300.99 0)
+			(hide yes)
+			(show_name no)
+			(do_not_autoplace no)
+			(effects
+				(font
+					(size 1.27 1.27)
+				)
+			)
+		)
 		(pin "16"
 		)
@@
 			)
 		)
-		(property "Footprint" ""
+		(property "Footprint" "Connector_USB:USB_C_Receptacle_GCT_USB4105-xx-A_16P_TopMnt_Horizontal"
 			(at 31.75 69.85 0)
 			(hide yes)
@@
 			)
 		)
-		(property "Footprint" "Package_DFN_QFN:QFN-48-1EP_6x6mm_P0.4mm_EP4.6x4.6mm"
+		(property "Footprint" "Package_DFN_QFN:QFN-48-1EP_6x6mm_P0.4mm_EP4.6x4.6mm_ThermalVias"
 			(at 472.44 464.82 0)
 			(hide yes)
@@
 			)
 		)
-		(property "Datasheet" "https://docs.nordicsemi.com/bundle/ps_nrf54L15"
+		(property "Datasheet" "https://docs.nordicsemi.com/bundle/ps_nrf54L10"
 			(at 472.44 467.36 0)
 			(hide yes)
@@
 			)
 		)
-		(property "MPN" ""
+		(property "MPN" "NRF54L10-QFAA-R7"
 			(at 472.44 393.7 0)
 			(hide yes)
@@
 			)
 		)
+		(property "Dielectric" ""
+			(at 472.44 393.7 0)
+			(hide yes)
+			(show_name no)
+			(do_not_autoplace no)
+			(effects
+				(font
+					(size 1.27 1.27)
+				)
+			)
+		)
+		(property "Tolerance" ""
+			(at 472.44 393.7 0)
+			(hide yes)
+			(show_name no)
+			(do_not_autoplace no)
+			(effects
+				(font
+					(size 1.27 1.27)
+				)
+			)
+		)
+		(property "Voltage" ""
+			(at 472.44 393.7 0)
+			(hide yes)
+			(show_name no)
+			(do_not_autoplace no)
+			(effects
+				(font
+					(size 1.27 1.27)
+				)
+			)
+		)
+		(property "Type" ""
+			(at 472.44 393.7 0)
+			(hide yes)
+			(show_name no)
+			(do_not_autoplace no)
+			(effects
+				(font
+					(size 1.27 1.27)
+				)
+			)
+		)
+		(property "LCSC Part" "C44800139"
+			(at 472.44 393.7 0)
+			(hide yes)
+			(show_name no)
+			(do_not_autoplace no)
+			(effects
+				(font
+					(size 1.27 1.27)
+				)
+			)
+		)
 		(pin "34"
 		)
@@
 			)
 		)
-		(property "Value" "BQ25713RSNT"
+		(property "Value" "BQ25713RSNR"
 			(at 156.21 499.11 0)
 			(show_name no)
@@
 			)
 		)
-		(property "MPN" ""
+		(property "MPN" "BQ25713RSNR"
 			(at 123.19 506.73 0)
 			(hide yes)
@@
 			)
 		)
+		(property "Dielectric" ""
+			(at 123.19 506.73 0)
+			(hide yes)
+			(show_name no)
+			(do_not_autoplace no)
+			(effects
+				(font
+					(size 1.27 1.27)
+				)
+			)
+		)
+		(property "Tolerance" ""
+			(at 123.19 506.73 0)
+			(hide yes)
+			(show_name no)
+			(do_not_autoplace no)
+			(effects
+				(font
+					(size 1.27 1.27)
+				)
+			)
+		)
+		(property "Voltage" ""
+			(at 123.19 506.73 0)
+			(hide yes)
+			(show_name no)
+			(do_not_autoplace no)
+			(effects
+				(font
+					(size 1.27 1.27)
+				)
+			)
+		)
+		(property "Type" ""
+			(at 123.19 506.73 0)
+			(hide yes)
+			(show_name no)
+			(do_not_autoplace no)
+			(effects
+				(font
+					(size 1.27 1.27)
+				)
+			)
+		)
+		(property "LCSC Part" "C2878935"
+			(at 123.19 506.73 0)
+			(hide yes)
+			(show_name no)
+			(do_not_autoplace no)
+			(effects
+				(font
+					(size 1.27 1.27)
+				)
+			)
+		)
 		(pin "28"
 		)
@@
 			)
 		)
-		(property "Value" "6.65k"
+		(property "Value" "5.6k"
 			(at 31.75 383.5399 0)
 			(show_name no)
@@
 			(at 29.21 382.27 0)
 			(hide yes)
+			(show_name no)
+			(do_not_autoplace no)
+			(effects
+				(font
+					(size 1.27 1.27)
+				)
+			)
+		)
+		(property "Dielectric" ""
+			(at 29.21 382.27 0)
+			(hide yes)
+			(show_name no)
+			(do_not_autoplace no)
+			(effects
+				(font
+					(size 1.27 1.27)
+				)
+			)
+		)
+		(property "Tolerance" "1%"
+			(at 29.21 382.27 0)
+			(hide yes)
+			(show_name no)
+			(do_not_autoplace no)
+			(effects
+				(font
+					(size 1.27 1.27)
+				)
+			)
+		)
+		(property "Voltage" ""
+			(at 29.21 382.27 0)
+			(hide yes)
+			(show_name no)
+			(do_not_autoplace no)
+			(effects
+				(font
+					(size 1.27 1.27)
+				)
+			)
+		)
+		(property "Type" ""
+			(at 29.21 382.27 0)
+			(hide yes)

Commit message: eeprom
Parts:
- R3: value 383k -> 390k; footprint (none) -> PCM_JLCPCB:R_0603
- R4: value 220k -> 240k
Changed lines of the file:
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@@
 			)
 		)
-		(property "Value" "383k"
+		(property "Value" "390k"
 			(at 68.58 549.9099 0)
 			(show_name no)
@@
 			)
 		)
-		(property "Footprint" ""
+		(property "Footprint" "PCM_JLCPCB:R_0603"
 			(at 64.262 548.64 90)
 			(hide yes)
@@
 			)
 		)
-		(property "Value" "220k"
+		(property "Value" "240k"
 			(at 68.58 560.0699 0)
 			(show_name no)

Commit message: update
Parts:
- R62, R9: footprint (none) -> Resistor_SMD:R_0805_2012Metric; LCSC Part (none) -> C17414
Changed lines of the file:
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@@
 			)
 		)
-		(property "Footprint" ""
+		(property "Footprint" "Resistor_SMD:R_0805_2012Metric"
 			(at 108.458 533.4 90)
 			(hide yes)
@@
 			)
 		)
+		(property "LCSC Part" "C17414"
+			(at 106.68 533.4 0)
+			(hide yes)
+			(show_name no)
+			(do_not_autoplace no)
+			(effects
+				(font
+					(size 1.27 1.27)
+				)
+			)
+		)
 		(pin "1"
 		)
@@
 			)
 		)
-		(property "Footprint" ""
+		(property "Footprint" "Resistor_SMD:R_0805_2012Metric"
 			(at 99.568 530.86 90)
 			(hide yes)
@@
 			(at 97.79 530.86 0)
 			(hide yes)
+			(show_name no)
+			(do_not_autoplace no)
+			(effects
+				(font
+					(size 1.27 1.27)
+				)
+			)
+		)
+		(property "LCSC Part" "C17414"
+			(at 97.79 530.86 0)
+			(hide yes)

Commit message: a
Parts:
- removed IC1: CAV24C256WE-GT3, symbol CAV24C256WE-GT3:CAV24C256WE-GT3
- added U4: AT24C256C-SSHL-T, AT24C256C-SSHL-T:SOIC127P600X175-8N, symbol AT24C256C-SSHL-T:AT24C256C-SSHL-T
- Q1, Q2, Q3, Q4: footprint footprints:CSD17308Q3 -> (none); MPN CSD17308Q3 -> (none)
- Q5: footprint Package_TO_SOT_SMD:SOT-23 -> (none); MPN CSD25404Q3 -> (none)
Connections:
- net GND: now also U4.1 (A0), U4.2 (A1), U4.3 (A2), U4.4 (GND), U4.7 (WP)
- net OUTPUT_LDO_3V3: now also U4.8 (VCC)
- net OUTPUT_SCL1: now also U4.6 (SCL)
- net OUTPUT_SDA1: now also U4.5 (SDA)
Other:
- moved on the sheet: R15, R16

Commit message: a
Parts:
- added H14: eSDA, TestPoint:TestPoint_THTPad_D2.5mm_Drill1.2mm, symbol Mechanical:MountingHole_Pad
- added H17: eSCL, TestPoint:TestPoint_THTPad_D2.5mm_Drill1.2mm, symbol Mechanical:MountingHole_Pad
- U3: footprint footprints:RSM32_TEX -> footprints:VQFN-32_L4.0-W4.0-P0.40-TL-EP1.4
- U4: LCSC Part (none) -> C6482
Connections:
- net CHGND: now also C48.1, J3.GND, R40.2, R41.1, U3.23 (PTC), U3.24 (PTCEN), U3.7 (NC)
- net GND: now also U3.14 (NC), U3.33 (EPAD); no longer U3.23 (PTC), U3.24 (PTCEN), U3.HTAB (EPAD)
- net OUTPUT_SCL1: now also H17.1
- net OUTPUT_SDA1: now also H14.1

Commit message: crystal
Parts:
- removed Y1: 32Mhz, Crystal:Crystal_SMD_2016-4Pin_2.0x1.6mm, symbol Device:Crystal
- added X1: XTM20032000DT00351005, CRYSTAL-SMD_4P-L2.0-W1.6-BL-A, symbol C37635332-XTM20032000DT00351005:XTM20032000DT00351005
Connections:
- net GND: now also X1.2 (GND), X1.4 (GND)
- net at U5.35 (XC2): now also X1.3
- net at U5.34 (XC1): now also X1.1
Other:
- note removed: "NOTE: double check crystal pins 13 might be crystal 24 ground"

Commit message: a
Parts:
- removed C2: 100pF, Capacitor_SMD:C_0603_1608Metric, symbol Device:C
- removed C65: 10uF, Capacitor_SMD:C_1206_3216Metric, symbol Device:C
- removed D12, D13: D_TVS, symbol Device:D_TVS
- removed H12: iBAT, symbol Mechanical:MountingHole_Pad
- removed J1, J4: USB_C_Receptacle, Connector_USB:USB_C_Receptacle_GCT_USB4105-xx-A_16P_TopMnt_Horizontal, symbol Connector:USB_C_Receptacle
- removed R6: 30k, Resistor_SMD:R_0402_1005Metric, symbol Device:R
- added C89, C91: 4.7uF, Capacitor_SMD:C_1206_3216Metric, symbol Device:C
- added C90, C92: 100nF, Capacitor_SMD:C_0603_1608Metric, symbol Device:C
- added C93: 10uF, Capacitor_SMD:C_0402_1005Metric, symbol Device:C
- added J2, J4: USB_C_Receptacle_USB2.0_16P, footprints:USB-C-SMD_TYPE-C16PIN, symbol Connector:USB_C_Receptacle_USB2.0_16P
- C10, C11, C13, C4, C6, C8: LCSC Part (none) -> C440198
- C15: footprint Capacitor_SMD:C_0603_1608Metric -> Capacitor_SMD:C_0805_2012Metric; LCSC Part (none) -> C13967
- C25, C26, C31, C35, C37, C45, C46, C47, C48, C55, C61, C62, C9: LCSC Part (none) -> C14663; MPN (none) -> CC0603KRX7R9BB104
- C28, C30: LCSC Part (none) -> C1664; MPN (none) -> CL10C331JB8NNNC
- C33, C57: footprint Capacitor_SMD:C_0402_1005Metric -> Capacitor_SMD:C_0603_1608Metric; LCSC Part (none) -> C14663; MPN (none) -> CC0603KRX7R9BB104
- C41: LCSC Part (none) -> C1623
- C42: footprint Capacitor_SMD:C_0603_1608Metric -> Capacitor_SMD:C_0402_1005Metric; LCSC Part (none) -> C307331; MPN (none) -> CL05B104KB54PNC
- C44: footprint Capacitor_SMD:C_0402_1005Metric -> (none); LCSC Part (none) -> C15525
- C51, C77, C78, C79: footprint Capacitor_SMD:C_0201_0603Metric -> Capacitor_SMD:C_0603_1608Metric; MPN (none) -> CC0603KRX7R9BB104
- C52, C60: LCSC Part (none) -> C14663; MPN (none) -> CC0603KRX7R9BB104; now fitted
- C71: footprint Capacitor_SMD:C_1206_3216Metric -> Capacitor_SMD:C_0805_2012Metric; LCSC Part (none) -> C440198
- C75: footprint (none) -> Capacitor_SMD:C_0402_1005Metric; LCSC Part (none) -> C15525
- C76: value 10uF -> 4.7uF
- D1, D3, D7, D8, D9: LCSC Part (none) -> C2290
- FB1: LCSC Part (none) -> C14709; MPN (none) -> BLM18PG121SN1D
- L2: LCSC Part (none) -> C5339435; MPN (none) -> XR0640-4R7M
- R1, R31: value 3.9 -> 3.7; footprint (none) -> Capacitor_SMD:C_0805_2012Metric; LCSC Part (none) -> 0805W8F470KT5E
- R13: LCSC Part (none) -> C105362
- R19, R22, R25, R29: footprint (none) -> Resistor_SMD:R_0805_2012Metric; LCSC Part (none) -> C17521; MPN (none) -> 0805W8F220KT5E
- R2, R23, R26: LCSC Part (none) -> C25077
- R20: LCSC Part (none) -> C22961
- R21: LCSC Part (none) -> C31850
- R27: footprint (none) -> Resistor_SMD:R_0402_1005Metric; LCSC Part (none) -> C25077
- R30: footprint Resistor_SMD:R_2010_5025Metric -> Resistor_SMD:R_1206_3216Metric; LCSC Part (none) -> C105362; Tolerance (none) -> 1%; Voltage (none) -> 50mV
- R40, R43: LCSC Part (none) -> C22775
- R41: value 0.001 -> 1m; footprint Resistor_SMD:R_1210_3225Metric -> Resistor_SMD:R_1206_3216Metric; LCSC Part (none) -> C7467246; Tolerance (none) -> 50 ppm
- R5: footprint (none) -> Resistor_SMD:R_0603_1608Metric; LCSC Part (none) -> C321717; Tolerance (none) -> 3%
- R65: footprint (none) -> Resistor_SMD:R_0402_1005Metric; LCSC Part (none) -> C25077; MPN (none) -> 0402WGF100JTCE
- R69: Power_Rating 0.5W -> 0.25W
- R7: LCSC Part (none) -> C25741
- R8: LCSC Part (none) -> C25774
- X1: value XTM20032000DT00351005 -> 32MHz; MPN (none) -> XTM20032000DT00351005
Connections:
- net BMS_SRP is gone; now on net BMS_SRN: C52.1, C57.1, C60.1, R40.1, U3.8 (SRP)
- net CC1_IN: now also J4.A5 (CC1)
- net CC1_OUT: now also J2.A5 (CC1)
- net CC2_IN: now also J4.B5 (CC2)
- net CC2_OUT: now also J2.B5 (CC2)
- net DM_OUT: now also J2.A7 (D-), J2.B7 (D-)
- net DP_OUT: now also J2.A6 (D+), J2.B6 (D+)
- net GND: now also C89.2, C90.2, C91.2, C92.2, C93.2, J2.A1 (GND), J2.A12 (GND), J2.B1 (GND), J2.B12 (GND), J2.SH (SHIELD), J4.A1 (GND), J4.A12 (GND), J4.B1 (GND), J4.B12 (GND), J4.SH (SHIELD)
- net PD_LDO_3V3: now also C93.1
- net VBUS_IN: now also J4.A4 (VBUS), J4.A9 (VBUS), J4.B4 (VBUS), J4.B9 (VBUS)
- net VBUS_OUT: now also J2.A4 (VBUS), J2.A9 (VBUS), J2.B4 (VBUS), J2.B9 (VBUS)
- net at U1.21 (LDO_5V): now also C89.1, C90.1
- net at U1.7 (LDO_1V5): now also C91.1, C92.1
- no-connect marks 74 -> 56
Other:
- note added: "1.83mA max"
- note added: "current sense calc ((3*0.01)^2)/0.01"
- note added: "place as close to batt 1N"
- moved on the sheet: C1, C10, C11, C12, C13, C14, C15, C16, C17, C18, C19, C20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

Commit message: update naming
Parts:
- C2: renamed from C1; footprint Capacitor_SMD:C_0805_2012Metric -> Resistor_SMD:R_0603_1608Metric; LCSC Part (none) -> C15849
- C4: renamed from C5; footprint Capacitor_SMD:C_0805_2012Metric -> Capacitor_SMD:C_0603_1608Metric; LCSC Part (none) -> C15849
- C52: renamed from C32; footprint Capacitor_SMD:C_0402_1005Metric -> Capacitor_SMD:C_0603_1608Metric; LCSC Part (none) -> C15849
- renumbered C41 to C1, C8 to C10, C23 to C11, C10 to C12, C66 to C13, C7 to C14, C25 to C15, C11 to C16, C89 to C17, C68 to C18, C9 to C19, C12 to C20, C67 to C21, C13 to C22, C14 to C23, C55 to C24, C90 to C25, C91 to C26, C70 to C27, C69 to C28, C15 to C29, C92 to C30, C93 to C31, C71 to C32, C16 to C33, C75 to C34, C76 to C35, C17 to C36, C18 to C37, C74 to C38, C19 to C39, C20 to C40, C30 to C41, C28 to C42, C72 to C43, C73 to C44, C21 to C45, C24 to C46, C22 to C47, C26 to C48, C34 to C49, C42 to C5, C35 to C50, C80 to C51, C81 to C53, C37 to C54, C33 to C55, C82 to C56, C38 to C57, C83 to C58, C39 to C59, C4 to C6, C31 to C60, C84 to C61, C27 to C62, C85 to C63, C29 to C64, C36 to C65, C86 to C66, C87 to C67, C88 to C68, C79 to C69, C63 to C7, C78 to C70, C77 to C71, C44 to C72, C51 to C73, C54 to C74, C50 to C75, C40 to C76, C58 to C77, C49 to C78, C59 to C79, C6 to C8, C61 to C80, C53 to C81, C43 to C82, C62 to C83, C56 to C84, C45 to C85, C46 to C86, C47 to C87, C48 to C88, C52 to C89, C64 to C9, C57 to C90, C60 to C91, D21 to D1, D1 to D10, D8 to D11, D3 to D12, D9 to D13, D15 to D14, D4 to D2, D2 to D3, D5 to D4, D6 to D5, D11 to D6, D10 to D7, D14 to D8, D7 to D9, H13 to H1, H6 to H10, H4 to H11, H3 to H12, H7 to H13, H11 to H14, H1 to H15, H2 to H16, H16 to H2, H15 to H3, H10 to H4, H8 to H5, H9 to H6, H14 to H7, H17 to H8, H5 to H9, J4 to J1, L8 to L5, R69 to R1, R4 to R10, R54 to R11, R55 to R12, R56 to R13, R57 to R14, R20 to R15, R21 to R16, R9 to R17, R58 to R18, R59 to R19, R7 to R2, R62 to R20, R10 to R21, R60 to R22, R61 to R23, R11 to R24, R12 to R25, R18 to R26, R13 to R27, R14 to R28, R17 to R29, R8 to R3, R19 to R30, R22 to R31, R27 to R32, R28 to R33, R23 to R34, R24 to R35, R26 to R36, R30 to R37, R15 to R38, R16 to R39, R1 to R4, R25 to R40, R29 to R41, R34 to R42, R32 to R43, R66 to R44, R33 to R45, R42 to R46, R44 to R47, R45 to R48, R46 to R49, R65 to R5, R47 to R50, R36 to R51, R37 to R52, R38 to R53, R39 to R54, R48 to R55, R35 to R56, R50 to R57, R51 to R58, R49 to R59, R31 to R6, R52 to R60, R40 to R61, R41 to R62, R53 to R63, R43 to R64, R2 to R7, R5 to R8, R3 to R9, SW3 to SW1, SW1 to SW2, SW2 to SW3, U2 to U1, U1 to U2, U6 to U3, U3 to U6
