File: pcb/FindMyCharger.kicad_sch (KiCad schematic)
At the start: 211 parts, among them J1 USB_C_Receptacle_USB2.0_16P, J2 Battery_Connector, J3 USB_C_Receptacle_USB2.0_16P, Q1 Q_PMOS, Q2 Q_NMOS, Q3 Q_NMOS, Q4 Q_NMOS, Q5 Q_NMOS, Q6 Q_NMOS, Q7 Q_PMOS, Q8 Q_NMOS, Q9 Q_NMOS, SW1 SW_Push, SW2 SW_Push, SW3 SW_Push, U1 TPS25730DREFR, U2 BQ25713RSNR, U3 nRF54L10-QFXX, U4 BQ4050RSMR, U5 TPS25762DQRQLRQ1, U6 AT24C256C-SSHL-T, X1 32MHz

Commit message: sch
Parts:
- Q1: MPN FDN358P -> (none)
- Q2, Q3: footprint (none) -> footprints:QNM30N20AJ-PDFN-8L_L3.3-W3.3-P0.65-BL_XINFEIHONG_FH1404G6; LCSC Part (none) -> C54300927; MPN Si7116DN -> QNM30N20AJ
- Q4: footprint Package_TO_SOT_SMD:SOT-23 -> footprints:QNM30N20AJ-PDFN-8L_L3.3-W3.3-P0.65-BL_XINFEIHONG_FH1404G6; LCSC Part C22379475 -> C54300927; MPN 2N7002K -> QNM30N20AJ
- Q5, Q6, Q8, Q9: footprint (none) -> footprints:QNM30N20AJ-PDFN-8L_L3.3-W3.3-P0.65-BL_XINFEIHONG_FH1404G6; LCSC Part (none) -> C54300927; MPN (none) -> QNM30N20AJ
Changed lines of the file:
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@@
 			)
 		)
-		(property "Footprint" "Package_TO_SOT_SMD:SOT-23"
+		(property "Footprint" "footprints:QNM30N20AJ-PDFN-8L_L3.3-W3.3-P0.65-BL_XINFEIHONG_FH1404G6"
 			(at 303.53 160.02 0)
 			(hide yes)
@@
 			)
 		)
-		(property "MPN" "2N7002K"
+		(property "MPN" "QNM30N20AJ"
 			(at 308.61 157.48 0)
 			(hide yes)
@@
 			)
 		)
-		(property "LCSC Part" "C22379475"
+		(property "LCSC Part" "C54300927"
 			(at 308.61 157.48 0)
 			(hide yes)
@@
 			)
 		)
-		(property "Footprint" ""
+		(property "Footprint" "footprints:QNM30N20AJ-PDFN-8L_L3.3-W3.3-P0.65-BL_XINFEIHONG_FH1404G6"
 			(at 276.86 149.86 0)
 			(hide yes)
@@
 			)
 		)
-		(property "MPN" "Si7116DN"
+		(property "MPN" "QNM30N20AJ"
 			(at 279.4 154.94 0)
 			(hide yes)
@@
 			)
 		)
+		(property "LCSC Part" "C54300927"
+			(at 124.46 434.34 0)
+			(show_name no)
+			(do_not_autoplace no)
+			(effects
+				(font
+					(size 1.27 1.27)
+				)
+			)
+		)
 		(pin "D"
 		)
@@
 			)
 		)
-		(property "Footprint" ""
+		(property "Footprint" "footprints:QNM30N20AJ-PDFN-8L_L3.3-W3.3-P0.65-BL_XINFEIHONG_FH1404G6"
 			(at 615.95 46.99 0)
 			(hide yes)
@@
 			)
 		)
-		(property "MPN" ""
+		(property "MPN" "QNM30N20AJ"
 			(at 613.41 52.07 0)
 			(hide yes)
@@
 			)
 		)
+		(property "LCSC Part" "C54300927"
+			(at 665.48 665.48 0)
+			(show_name no)
+			(do_not_autoplace no)
+			(effects
+				(font
+					(size 1.27 1.27)
+				)
+			)
+		)
 		(pin "D"
 		)
@@
 			)
 		)
-		(property "MPN" "FDN358P"
+		(property "MPN" ""
 			(at 255.27 146.05 0)
 			(hide yes)
@@
 			)
 		)
-		(property "Footprint" ""
+		(property "Footprint" "footprints:QNM30N20AJ-PDFN-8L_L3.3-W3.3-P0.65-BL_XINFEIHONG_FH1404G6"
 			(at 248.92 149.86 0)
 			(hide yes)
@@
 			)
 		)
-		(property "MPN" "Si7116DN"
+		(property "MPN" "QNM30N20AJ"
 			(at 246.38 154.94 0)
 			(hide yes)
@@
 			)
 		)
+		(property "LCSC Part" "C54300927"
+			(at 246.38 154.94 0)
+			(hide yes)
+			(show_name no)
+			(do_not_autoplace no)
+			(effects
+				(font
+					(size 1.27 1.27)
+				)
+			)
+		)
 		(pin "D"
 		)
@@
 			)
 		)
-		(property "Footprint" ""
+		(property "Footprint" "footprints:QNM30N20AJ-PDFN-8L_L3.3-W3.3-P0.65-BL_XINFEIHONG_FH1404G6"
 			(at 528.32 46.99 0)
 			(hide yes)
@@
 			)
 		)
-		(property "MPN" ""
+		(property "MPN" "QNM30N20AJ"
 			(at 530.86 52.07 0)
 			(hide yes)
@@
 			)
 		)
+		(property "LCSC Part" "C54300927"
+			(at 530.86 52.07 0)
+			(hide yes)
+			(show_name no)
+			(do_not_autoplace no)
+			(effects
+				(font
+					(size 1.27 1.27)
+				)
+			)
+		)
 		(pin "G"
 		)
@@
 			)
 		)
-		(property "Footprint" ""
+		(property "Footprint" "footprints:QNM30N20AJ-PDFN-8L_L3.3-W3.3-P0.65-BL_XINFEIHONG_FH1404G6"
 			(at 546.1 52.07 0)
 			(hide yes)
@@
 			)
 		)
-		(property "MPN" ""
+		(property "MPN" "QNM30N20AJ"
 			(at 541.02 54.61 0)
 			(hide yes)
@@
 			)
 		)
+		(property "LCSC Part" "C54300927"
+			(at 0 0 0)
+			(hide yes)
+			(show_name no)
+			(do_not_autoplace no)
+			(effects
+				(font
+					(size 1.27 1.27)
+				)
+			)
+		)
 		(pin "G"
 		)
@@
 			)
 		)
-		(property "Footprint" ""
+		(property "Footprint" "footprints:QNM30N20AJ-PDFN-8L_L3.3-W3.3-P0.65-BL_XINFEIHONG_FH1404G6"
 			(at 598.17 52.07 0)
 			(hide yes)
@@
 			)
 		)
-		(property "MPN" ""
+		(property "MPN" "QNM30N20AJ"
 			(at 603.25 54.61 0)
 			(hide yes)
@@
 			(show_name no)
 			(do_not_autoplace no)
+			(effects
+				(font
+					(size 1.27 1.27)
+				)
+			)
+		)
+		(property "LCSC Part" "C54300927"
+			(at 1206.5 0 0)
+			(show_name no)
+			(do_not_autoplace no)

Commit message: updated footprint
Parts:
- Q2: renamed from Q1; footprint Package_TO_SOT_SMD:SOT-23 -> footprints:ZC015P2G-POWERTDFN-8_L3.1-W3.1-P0.65-LS3.3-BL; LCSC Part (none) -> C53433530
- Q9: renamed from Q7; footprint (none) -> footprints:ZC015P2G-POWERTDFN-8_L3.1-W3.1-P0.65-LS3.3-BL; LCSC Part (none) -> C53433530
- SW1: renamed from SW2; footprint (none) -> Button_Switch_THT:SW_PUSH_6mm
- SW2: renamed from SW1; footprint (none) -> Button_Switch_THT:SW_PUSH_6mm
- SW3: footprint (none) -> Button_Switch_THT:SW_PUSH_6mm
- renumbered C34 to C1, C5 to C10, C48 to C11, C44 to C12, C63 to C13, C7 to C14, C11 to C15, C49 to C16, C56 to C17, C1 to C18, C8 to C19, C35 to C2, C12 to C20, C50 to C21, C57 to C22, C58 to C23, C9 to C24, C10 to C25, C62 to C26, C13 to C27, C14 to C28, C42 to C29, C2 to C3, C43 to C30, C45 to C31, C46 to C32, C51 to C33, C47 to C34, C52 to C35, C22 to C36, C86 to C37, C23 to C38, C87 to C39, C36 to C4, C24 to C40, C25 to C41, C26 to C42, C83 to C43, C55 to C44, C27 to C45, C60 to C46, C69 to C47, C84 to C48, C78 to C49, C3 to C5, C41 to C50, C70 to C51, C85 to C52, C39 to C53, C79 to C54, C80 to C55, C81 to C56, C40 to C57, C28 to C58, C29 to C59, C37 to C6, C61 to C60, C59 to C61, C82 to C62, C88 to C63, C30 to C64, C31 to C65, C53 to C67, C15 to C68, C71 to C69, C4 to C7, C33 to C70, C16 to C71, C64 to C72, C68 to C73, C72 to C74, C32 to C75, C17 to C76, C73 to C77, C18 to C78, C74 to C79, C38 to C8, C19 to C80, C54 to C81, C75 to C82, C20 to C83, C65 to C84, C76 to C85, C21 to C86, C77 to C87, C67 to C88, C6 to C9, D4 to D2, D2 to D3, D3 to D4, D6 to D5, D9 to D6, D5 to D7, D7 to D9, H9 to H1, H12 to H10, H10 to H12, H15 to H13, H3 to H14, H14 to H15, H1 to H2, H2 to H3, H5 to H4, H8 to H5, H4 to H6, H6 to H8, H13 to H9, L2 to L1, L4 to L2, L5 to L4, L1 to L5, Q2 to Q1, Q8 to Q6, Q9 to Q7, Q6 to Q8, R44 to R10, R47 to R11, R45 to R12, R48 to R13, R12 to R14, R10 to R15, R15 to R18, R27 to R19, R5 to R2, R28 to R20, R29 to R21, R30 to R22, R18 to R23, R19 to R24, R11 to R25, R9 to R26, R14 to R27, R35 to R28, R42 to R29, R2 to R3, R13 to R30, R36 to R31, R59 to R32, R63 to R33, R31 to R34, R33 to R35, R62 to R36, R65 to R37, R53 to R38, R41 to R39, R6 to R4, R54 to R40, R24 to R41, R55 to R42, R22 to R43, R20 to R44, R23 to R45, R64 to R46, R43 to R47, R34 to R48, R38 to R49, R3 to R5, R49 to R50, R32 to R51, R50 to R52, R37 to R53, R40 to R54, R25 to R55, R21 to R56, R56 to R57, R57 to R58, R26 to R59, R7 to R6, R58 to R60, R60 to R61, R61 to R62, R39 to R63, R51 to R64, R52 to R65, R4 to R7, R46 to R9, U3 to U1, U1 to U2, U4 to U3, U2 to U4
Connections:
- net INPUT_IBAT: no longer names the net of U4.9 (IBAT)
- net INPUT_PSYS: no longer names the net of U4.10 (PSYS)
- no-connect marks 57 -> 59

Commit message: excl debug/pads from bom
Parts:
- AE1, J2: now left out of the parts list
- C17: LCSC Part C435397 -> C1552; MPN GJM0335C1E1R5WB01 -> (none)
- C24, C25, C62, C63, C81: footprint Resistor_SMD:R_0402_1005Metric -> Capacitor_SMD:C_0402_1005Metric
- C36: LCSC Part 10uF1 -> C440198
- C44: LCSC Part (none) -> C1562
- C46: LCSC Part (none) -> C696873
- C60: footprint Capacitor_SMD:C_0402_1005Metric -> Capacitor_SMD:C_0603_1608Metric; LCSC Part (none) -> C1630
- C61: LCSC Part (none) -> C1548
- C68, C71, C76, C78, C80, C83, C86: footprint Capacitor_SMD:C_0603_1608Metric -> Capacitor_SMD:C_0805_2012Metric; LCSC Part (none) -> C440198
- R1: now not fitted
- R10, R11: footprint Capacitor_SMD:C_0402_1005Metric -> Resistor_SMD:R_0402_1005Metric_Pad0.72x0.64mm_HandSolder; LCSC Part (none) -> C25087
- R12, R13, R19, R20, R21, R22, R28, R31: footprint Capacitor_SMD:C_0402_1005Metric -> Resistor_SMD:R_0402_1005Metric
- R14, R18, R25: LCSC Part C384386 -> C52209954
- R43, R45: value 4.99 -> 4.7; footprint Capacitor_SMD:C_0402_1005Metric -> Resistor_SMD:R_0805_2012Metric; LCSC Part (none) -> C17675
- R53: footprint PCM_JLCPCB:R_0603 -> Resistor_SMD:R_0603_1608Metric
- R9: LCSC Part C21190 -> C11702
- U2: LCSC Part (none) -> C22438973
- U3: LCSC Part (none) -> C157570
Connections:
- no-connect marks 59 -> 57
Other:
- note added: "Low input filter"

Commit message: finished mapping
Parts:
- removed R6: 40.2k, Resistor_SMD:R_0805_2012Metric, symbol Device:R
- added R66: 40.2k, Resistor_SMD:R_0603_1608Metric, symbol Device:R
- C50, C73: footprint Capacitor_SMD:C_0805_2012Metric -> Capacitor_SMD:C_0603_1608Metric; LCSC Part C13967 -> C1623
- C67, C70: footprint Capacitor_SMD:C_0603_1608Metric -> Capacitor_SMD:C_0402_1005Metric; LCSC Part C15849 -> C52923
- J1, J3: LCSC Part (none) -> C18357551
- L1: footprint Inductor_SMD:L_0603_1608Metric -> footprints:IND-SMD_L7.0-W6.6; LCSC Part (none) -> C5339435
- L2, L4: LCSC Part (none) -> C3911055
- L3: LCSC Part (none) -> C7216765
- R1: now left out of the parts list
- R43, R45: footprint Resistor_SMD:R_0805_2012Metric -> Resistor_SMD:R_0603_1608Metric; LCSC Part C17675 -> C23164
- R56: LCSC Part (none) -> C105362
Connections:
- net GND: now also J1.A1B12 (GND), J1.B1A12 (GND), J3.A1B12 (GND), J3.B1A12 (GND), R66.2; no longer J1.A1 (GND), J1.A12 (GND), J1.B1 (GND), J1.B12 (GND), J3.A1 (GND), J3.A12 (GND), J3.B1 (GND), J3.B12 (GND)
- net PD_ADCIN3: now also R66.1
- net VBUS_IN: now also J1.A4B9 (VBUS), J1.B4A9 (VBUS); no longer J1.A4 (VBUS), J1.A9 (VBUS), J1.B4 (VBUS), J1.B9 (VBUS)
- net VBUS_OUT: now also J3.A4B9 (VBUS), J3.B4A9 (VBUS); no longer J3.A4 (VBUS), J3.A9 (VBUS), J3.B4 (VBUS), J3.B9 (VBUS)

Commit message: dumped
Parts:
- SW3: footprint Button_Switch_THT:SW_PUSH_6mm -> Connector_Wire:SolderWire-0.127sqmm_1x02_P3.7mm_D0.48mm_OD1mm
Changed lines of the file:
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@@
 			)
 		)
-		(property "Footprint" "Button_Switch_THT:SW_PUSH_6mm"
+		(property "Footprint" "Connector_Wire:SolderWire-0.127sqmm_1x02_P3.7mm_D0.48mm_OD1mm"
 			(at 388.62 295.91 0)
 			(hide yes)

Commit message: rean
Parts:
- renumbered C18 to C1, C86 to C10, C7 to C11, C10 to C12, C9 to C13, C19 to C15, C36 to C16, C38 to C17, C40 to C18, C41 to C19, C3 to C2, C42 to C20, C45 to C21, C58 to C22, C59 to C23, C64 to C24, C65 to C25, C75 to C26, C24 to C27, C25 to C28, C70 to C29, C5 to C3, C15 to C30, C53 to C31, C57 to C32, C20 to C33, C50 to C34, C67 to C35, C81 to C36, C27 to C37, C28 to C38, C44 to C39, C68 to C4, C61 to C40, C46 to C41, C60 to C42, C1 to C43, C2 to C44, C4 to C45, C6 to C46, C8 to C47, C72 to C48, C84 to C49, C71 to C5, C66 to C50, C88 to C51, C29 to C52, C30 to C53, C12 to C54, C73 to C55, C31 to C56, C32 to C57, C34 to C58, C11 to C59, C76 to C6, C16 to C60, C21 to C61, C47 to C62, C51 to C63, C69 to C64, C74 to C65, C77 to C66, C79 to C67, C82 to C68, C85 to C69, C78 to C7, C87 to C70, C33 to C71, C35 to C72, C49 to C73, C54 to C74, C17 to C75, C22 to C76, C23 to C77, C55 to C78, C56 to C79, C80 to C8, C26 to C80, C62 to C81, C43 to C82, C48 to C83, C52 to C84, C13 to C85, C37 to C86, C39 to C87, C63 to C88, C83 to C9, D8 to D10, D6 to D11, D3 to D2, D4 to D3, D10 to D4, D11 to D5, D2 to D6, D5 to D8, H2 to H1, H8 to H10, H15 to H11, H7 to H12, H5 to H13, H13 to H14, H16 to H15, H1 to H16, H3 to H2, H14 to H3, H12 to H4, H11 to H5, H10 to H6, H9 to H7, H6 to H8, H4 to H9, J3 to J2, J2 to J3, L5 to L1, L6 to L2, L1 to L3, L3 to L4, L2 to L5, L4 to L6, Q5 to Q1, Q8 to Q2, Q9 to Q3, Q6 to Q4, Q7 to Q5, Q2 to Q6, Q1 to Q7, Q3 to Q8, Q4 to Q9, R44 to R1, R5 to R10, R7 to R11, R2 to R12, R4 to R13, R66 to R14, R8 to R15, R34 to R16, R51 to R17, R35 to R18, R48 to R19, R56 to R2, R53 to R20, R49 to R21, R63 to R22, R54 to R23, R39 to R24, R26 to R25, R47 to R26, R15 to R27, R25 to R28, R14 to R29, R43 to R3, R27 to R31, R18 to R32, R16 to R33, R17 to R34, R23 to R35, R24 to R36, R50 to R37, R52 to R38, R64 to R39, R45 to R4, R65 to R40, R19 to R41, R38 to R42, R40 to R43, R42 to R44, R20 to R45, R57 to R46, R21 to R47, R58 to R48, R22 to R49, R41 to R5, R60 to R50, R28 to R51, R31 to R52, R29 to R53, R10 to R54, R12 to R55, R9 to R56, R32 to R57, R61 to R58, R62 to R59, R55 to R6, R36 to R60, R33 to R61, R46 to R62, R11 to R63, R13 to R64, R37 to R65, R59 to R7, R1 to R8, R3 to R9, SW2 to SW1, SW3 to SW2, SW1 to SW3, U2 to U1, U4 to U2, U5 to U3, U1 to U4, U3 to U5

Commit message: a
Parts:
- removed R12: 0, Resistor_SMD:R_0603_1608Metric, symbol Device:R
- removed R8: DNP, Resistor_SMD:R_0603_1608Metric, symbol Device:R
Connections:
- net PD_ADCIN1 is gone; now on net GND: U1.2 (ADCIN1)

Commit message: a
Parts:
- removed H3: iCHG, TestPoint:TestPoint_Pad_D2.5mm, symbol Mechanical:MountingHole_Pad
Changed lines of the file:
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@@
 	)
 	(junction
-		(at 690.88 127)
-		(diameter 0)
-		(color 0 0 0 0)
-	)
-	(junction
 		(at 326.39 256.54)
 		(diameter 0)
@@
 	(wire
 		(pts
-			(xy 690.88 127) (xy 694.69 127)
-		)
-		(stroke
-			(width 0)
-			(type default)
-		)
-	)
-	(wire
-		(pts
 			(xy 125.73 243.84) (xy 132.08 243.84)
 		)
@@
 					(unit 1)
 				)
-			)
-		)
-	)
-	(symbol
-		(lib_id "Mechanical:MountingHole_Pad")
-		(at 697.23 127 270)
-		(unit 1)
-		(body_style 1)
-		(exclude_from_sim no)
-		(in_bom no)
-		(on_board yes)
-		(in_pos_files yes)
-		(dnp no)
-		(fields_autoplaced yes)
-		(property "Reference" "H3"
-			(at 701.04 125.7299 90)
-			(show_name no)
-			(do_not_autoplace no)
-			(effects
-				(font
-					(size 1.27 1.27)
-				)
-				(justify left)
-			)
-		)
-		(property "Value" "iCHG"
-			(at 701.04 128.2699 90)
-			(show_name no)
-			(do_not_autoplace no)
-			(effects
-				(font
-					(size 1.27 1.27)
-				)
-				(justify left)
-			)
-		)
-		(property "Footprint" "TestPoint:TestPoint_Pad_D2.5mm"
-			(at 697.23 127 0)
-			(hide yes)
-			(show_name no)
-			(do_not_autoplace no)
-			(effects
-				(font
-					(size 1.27 1.27)
-				)
-			)
-		)
-		(property "Datasheet" ""
-			(at 697.23 127 0)
-			(hide yes)
-			(show_name no)
-			(do_not_autoplace no)
-			(effects
-				(font
-					(size 1.27 1.27)
-				)
-			)
-		)
-		(property "Description" "Mounting Hole with connection"
-			(at 697.23 127 0)
-			(hide yes)
-			(show_name no)
-			(do_not_autoplace no)
-			(effects
-				(font
-					(size 1.27 1.27)
-				)
-			)
-		)
-		(pin "1"
-		)
-		(instances
-			(project "FindMyCharger"
-				(path "/263c00ee-f9a5-4919-b1d1-0dbcc4b9e7aa"
-					(reference "H3")
-					(unit 1)
-				)
