File: pcb/FindMyCharger.kicad_pcb (KiCad board)
At the start: 2 copper layers, 211 parts, among them J1 USB_C_Receptacle_USB2.0_16P, J2 Battery_Connector, J3 USB_C_Receptacle_USB2.0_16P, Q1 Q_NMOS, Q2 Q_PMOS, Q3 Q_NMOS, Q4 Q_NMOS, Q5 Q_NMOS, Q6 Q_NMOS, Q7 Q_NMOS, Q8 Q_NMOS, Q9 Q_PMOS, SW1 SW_Push, SW2 SW_Push, SW3 SW_Push, U1 nRF54L10-QFXX, U2 TPS25730DREFR, U3 BQ4050RSMR, U4 BQ25713RSNR, U5 TPS25762DQRQLRQ1, U6 AT24C256C-SSHL-T, X1 32MHz

Commit message: finished mapping
Parts:
- removed R6: 40.2k, Resistor_SMD:R_0805_2012Metric
- added R66: 40.2k, Resistor_SMD:R_0603_1608Metric, F.Cu at (48.2, 52.4)
- C50, C73: footprint Capacitor_SMD:C_0805_2012Metric -> Capacitor_SMD:C_0603_1608Metric
- C67, C70: footprint Capacitor_SMD:C_0603_1608Metric -> Capacitor_SMD:C_0402_1005Metric
- L1: footprint Inductor_SMD:L_0603_1608Metric -> footprints:IND-SMD_L7.0-W6.6
- R43, R45: footprint Resistor_SMD:R_0805_2012Metric -> Resistor_SMD:R_0603_1608Metric
- moved R15 65.2 mm to (29.4, 58.4)
- moved R29 65.2 mm to (29.4, 61.7)
- moved R44 65.2 mm to (29.4, 65.0)
- moved R56 65.2 mm to (29.4, 68.4)
- moved R60 65.2 mm to (29.4, 71.7)
- moved AE1 60.4 mm to (37.6, 29.0)
- moved C24 56.6 mm to (35.6, 70.9)
- moved C25 56.6 mm to (35.6, 72.9)
- moved C34 54.5 mm to (38.5, 70.9)
- moved C35 54.5 mm to (38.5, 72.9)
- moved C32 54.5 mm to (38.5, 67.0)
- moved C33 54.5 mm to (38.5, 68.9)
- moved C72 52.6 mm to (44.2, 72.9)
- moved C55 52.6 mm to (41.4, 70.9)
- moved C58 52.6 mm to (41.4, 72.9)
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Connections:
- J1 pad A1B12: (no net) -> GND
- J1 pad A4B9: (no net) -> VBUS_IN
- J1 pad B1A12: (no net) -> GND
- J1 pad B4A9: (no net) -> VBUS_IN
- J3 pad A1B12: (no net) -> GND
- J3 pad A4B9: (no net) -> VBUS_OUT
- J3 pad B1A12: (no net) -> GND
- J3 pad B4A9: (no net) -> VBUS_OUT

Commit message: pcbbb
Parts:
- removed AE1: Antenna, RF_Antenna:Texas_SWRA117D_2.4GHz_Right
- removed C1, C2, C4, C51, C54, C56, C8: 100nF, Capacitor_SMD:C_0603_1608Metric
- removed C10, C19, C36, C38, C40, C41, C42, C45, C68, C71, C76, C78, C80, C83, C86: 10uF, Capacitor_SMD:C_0805_2012Metric
- removed C11, C12, C21, C26: 2.2uF, Capacitor_SMD:C_0805_2012Metric
- removed C13, C22: 2pF, Capacitor_SMD:C_0201_0603Metric
- removed C14, C43, C77, C79, C9: 22uF, Capacitor_SMD:C_0805_2012Metric
- removed C15, C18, C6: 10uF, Capacitor_SMD:C_0402_1005Metric
- removed C16: 10nF, Capacitor_SMD:C_0201_0603Metric
- removed C17: 1.5pF, Capacitor_SMD:C_0201_0603Metric
- removed C20, C47, C49, C55: 4.7uF, Capacitor_SMD:C_0402_1005Metric
- removed C23: 0.3pF, Capacitor_SMD:C_0201_0603Metric
- removed C24, C25, C62, C63, C81: 330pF, Capacitor_SMD:C_0402_1005Metric
- removed C27, C28, C29, C3, C30, C31, C32, C33, C34, C35, C39, C48, C5, C52, C69, C7, C72, C74, C75, C84, C85, C87: 0.1uF, Capacitor_SMD:C_0402_1005Metric
- removed C37, C50, C73: 470nF, Capacitor_SMD:C_0603_1608Metric
- removed C44: 33pF, Capacitor_SMD:C_0402_1005Metric
- removed C46: 1.8nF, Capacitor_SMD:C_0402_1005Metric
- removed C53, C57: 33nF, Capacitor_SMD:C_0603_1608Metric
- removed C58: 10nF, Capacitor_SMD:C_0402_1005Metric
- removed C59, C66: 1nF, Capacitor_SMD:C_0402_1005Metric
- removed C60: 680pF, Capacitor_SMD:C_0603_1608Metric
- removed C61: 15pF, Capacitor_SMD:C_0402_1005Metric
- removed C64, C65: 47nF, Capacitor_SMD:C_0603_1608Metric
- removed C67, C70: 1uF, Capacitor_SMD:C_0402_1005Metric
- removed C82: 100uF, footprints:CAP-SMD_L7.3-W6.1_TCN4227M025R0100
- removed C88: 3.3nF, Capacitor_SMD:C_0402_1005Metric
- removed D1, D4: 30V, PCM_JLCPCB:D_SOT-23
- removed D10, D11, D2, D3: H5VU25U, PCM_JLCPCB:DFN2510-10_L2.5-W1.0-P0.50-BL
- removed D5, D6, D7, D8, D9: LED, LED_SMD:LED_0603_1608Metric
- removed FB1: 120, Inductor_SMD:L_0603_1608Metric
- removed H1: nSWDIO, TestPoint:TestPoint_THTPad_D2.5mm_Drill1.2mm
- removed H10: oSDA, TestPoint:TestPoint_THTPad_D2.5mm_Drill1.2mm
- removed H11: oSCL, TestPoint:TestPoint_THTPad_D2.5mm_Drill1.2mm
- removed H12: oIRQ, TestPoint:TestPoint_THTPad_D2.5mm_Drill1.2mm
- removed H13: eSDA, TestPoint:TestPoint_THTPad_D2.5mm_Drill1.2mm
- removed H14: iCHG, TestPoint:TestPoint_Pad_D2.5mm
- removed H15: eSCL, TestPoint:TestPoint_THTPad_D2.5mm_Drill1.2mm
- removed H16: GND, TestPoint:TestPoint_THTPad_2.5x2.5mm_Drill1.2mm
- removed H2: cSDA, TestPoint:TestPoint_THTPad_D2.5mm_Drill1.2mm
- removed H3: cSCL, TestPoint:TestPoint_THTPad_D2.5mm_Drill1.2mm
- removed H4: nRST, TestPoint:TestPoint_THTPad_D2.5mm_Drill1.2mm
- removed H5: nSWDCLK, TestPoint:TestPoint_THTPad_D2.5mm_Drill1.2mm
- removed H6: bSMBC, TestPoint:TestPoint_THTPad_D2.5mm_Drill1.2mm
- removed H7: bSMBD, TestPoint:TestPoint_THTPad_D2.5mm_Drill1.2mm
- removed H8: FUSE, TestPoint:TestPoint_Pad_D2.5mm
- removed H9: 3V3, TestPoint:TestPoint_THTPad_D2.5mm_Drill1.2mm
- removed J1, J3: USB_C_Receptacle_USB2.0_16P, footprints:USB-C-SMD_TYPE-C16PIN
- removed J2: Battery_Connector, footprints:BMS_4S_PAD
- removed L1, L6: 4.7uH, footprints:IND-SMD_L7.0-W6.6
- removed L2, L4: 3.5nH, Inductor_SMD:L_0201_0603Metric
- removed L3: 2.7nH, Inductor_SMD:L_0201_0603Metric
- removed L5: 2.2uH, footprints:IND-SMD_L7.1-W6.6
- removed Q1, Q3, Q4, Q5, Q6, Q7, Q8: Q_NMOS, footprints:QNM30N20AJ-PDFN-8L_L3.3-W3.3-P0.65-BL_XINFEIHONG_FH1404G6
- removed Q2, Q9: Q_PMOS, footprints:ZC015P2G-POWERTDFN-8_L3.1-W3.1-P0.65-LS3.3-BL
- removed R1: DNP, Resistor_SMD:R_0603_1608Metric
- removed R10, R11: 200, Resistor_SMD:R_0402_1005Metric_Pad0.72x0.64mm_HandSolder
- removed R12, R13, R19, R20, R21, R22, R23, R28, R31: 100, Resistor_SMD:R_0402_1005Metric
- removed R14, R18, R25: 10M, Resistor_SMD:R_0402_1005Metric
- removed R15: 300, Resistor_SMD:R_1206_3216Metric
- removed R16, R17, R24: 5.1k, Resistor_SMD:R_0402_1005Metric
- removed R2, R57: 0, Resistor_SMD:R_0603_1608Metric
- removed R26, R27, R3, R30, R34, R35, R47, R48, R8: 10k, Resistor_SMD:R_0805_2012Metric
- removed R29: 1m, Resistor_SMD:R_1206_3216Metric
- removed R32: 5.6k, Resistor_SMD:R_0402_1005Metric
- removed R33, R51, R55, R58, R59: 10, Resistor_SMD:R_0402_1005Metric
- removed R36, R4, R49, R54, R7: 220k, Resistor_SMD:R_0402_1005Metric
- removed R37: 22k, Resistor_SMD:R_0402_1005Metric
- removed R38, R40, R42, R46, R61, R62: 4.7k, Resistor_SMD:R_0402_1005Metric
- removed R39, R66: 40.2k, Resistor_SMD:R_0603_1608Metric
- removed R41: 1, Resistor_SMD:R_0402_1005Metric
- removed R43, R45: 4.7, Resistor_SMD:R_0603_1608Metric
- removed R44, R56, R60: 10m, Resistor_SMD:R_1206_3216Metric
- removed R5: 160k, Resistor_SMD:R_0603_1608Metric
- removed R50, R52, R64, R65: 2.2, Resistor_SMD:R_0805_2012Metric
- removed R53: 390k, Resistor_SMD:R_0603_1608Metric
- removed R63: 137k, Resistor_SMD:R_0603_1608Metric
- removed R9: 1k, Resistor_SMD:R_0603_1608Metric
- removed SW1, SW2, SW3: SW_Push, Button_Switch_THT:SW_PUSH_6mm
- removed TH1: 10k, Connector_Wire:SolderWire-0.127sqmm_1x02_P3.7mm_D0.48mm_OD1mm
- removed U1: nRF54L10-QFXX, Package_DFN_QFN:QFN-48-1EP_6x6mm_P0.4mm_EP4.6x4.6mm_ThermalVias
- removed U2: TPS25730DREFR, footprints:REF0038A-MFG
- removed U3: BQ4050RSMR, footprints:VQFN-32_L4.0-W4.0-P0.40-TL-EP1.4
- removed U4: BQ25713RSNR, footprints:RSN32_TEX
- removed U5: TPS25762DQRQLRQ1, footprints:RQL0029A-MFG
- removed U6: AT24C256C-SSHL-T, footprints:SOIC-8_L4.9-W3.9-P1.27-LS6.0-BL
- removed X1: 32MHz, footprints:CRYSTAL-SMD_4P-L2.0-W1.6-BL-A
Other:
- board text added: "18650"

Commit message: dumped
Parts:
- added AE1: Antenna, RF_Antenna:Texas_SWRA117D_2.4GHz_Right, F.Cu at (64.9, 81.6)
- added C1: 100nF, Capacitor_SMD:C_0603_1608Metric, F.Cu at (20.0, 61.0)
- added C10: 10uF, Capacitor_SMD:C_0805_2012Metric, F.Cu at (20.2, 25.0)
- added C11: 2.2uF, Capacitor_SMD:C_0805_2012Metric, F.Cu at (20.2, 28.0)
- added C12: 2.2uF, Capacitor_SMD:C_0805_2012Metric, F.Cu at (20.2, 31.0)
- added C13: 2pF, Capacitor_SMD:C_0201_0603Metric, F.Cu at (46.0, 26.7)
- added C14: 22uF, Capacitor_SMD:C_0805_2012Metric, F.Cu at (20.2, 34.0)
- added C15: 10uF, Capacitor_SMD:C_0402_1005Metric, F.Cu at (37.6, 50.4)
- added C16: 10nF, Capacitor_SMD:C_0201_0603Metric, F.Cu at (46.0, 28.4)
- added C17: 1.5pF, Capacitor_SMD:C_0201_0603Metric, F.Cu at (46.0, 30.2)
- added C18: 10uF, Capacitor_SMD:C_0402_1005Metric, F.Cu at (37.6, 52.4)
- added C19: 10uF, Capacitor_SMD:C_0805_2012Metric, F.Cu at (20.2, 37.1)
- added C2: 100nF, Capacitor_SMD:C_0603_1608Metric, F.Cu at (20.0, 63.5)
- added C20: 4.7uF, Capacitor_SMD:C_0402_1005Metric, F.Cu at (37.6, 54.4)
- added C21: 2.2uF, Capacitor_SMD:C_0805_2012Metric, F.Cu at (20.2, 40.1)
- added C22: 2pF, Capacitor_SMD:C_0201_0603Metric, F.Cu at (46.0, 31.9)
- added C23: 0.3pF, Capacitor_SMD:C_0201_0603Metric, F.Cu at (46.0, 33.7)
- added C24: 330pF, Capacitor_SMD:C_0402_1005Metric, F.Cu at (37.6, 56.3)
- added C25: 330pF, Capacitor_SMD:C_0402_1005Metric, F.Cu at (37.6, 58.3)
- added C26: 2.2uF, Capacitor_SMD:C_0805_2012Metric, F.Cu at (24.7, 22.0)
- added C27: 0.1uF, Capacitor_SMD:C_0402_1005Metric, F.Cu at (40.5, 42.6)
- added C28: 0.1uF, Capacitor_SMD:C_0402_1005Metric, F.Cu at (40.5, 44.5)
- added C29: 0.1uF, Capacitor_SMD:C_0402_1005Metric, F.Cu at (40.5, 46.5)
- added C3: 0.1uF, Capacitor_SMD:C_0402_1005Metric, F.Cu at (37.6, 42.6)
- added C30: 0.1uF, Capacitor_SMD:C_0402_1005Metric, F.Cu at (40.5, 48.5)
- added C31: 0.1uF, Capacitor_SMD:C_0402_1005Metric, F.Cu at (40.5, 50.4)
- added C32: 0.1uF, Capacitor_SMD:C_0402_1005Metric, F.Cu at (40.5, 52.4)
- added C33: 0.1uF, Capacitor_SMD:C_0402_1005Metric, F.Cu at (40.5, 54.4)
- added C34: 0.1uF, Capacitor_SMD:C_0402_1005Metric, F.Cu at (40.5, 56.3)
- added C35: 0.1uF, Capacitor_SMD:C_0402_1005Metric, F.Cu at (40.5, 58.3)
- added C36: 10uF, Capacitor_SMD:C_0805_2012Metric, F.Cu at (24.7, 25.0)
- added C37: 470nF, Capacitor_SMD:C_0603_1608Metric, F.Cu at (20.0, 71.1)
- added C38: 10uF, Capacitor_SMD:C_0805_2012Metric, F.Cu at (24.7, 28.0)
- added C39: 0.1uF, Capacitor_SMD:C_0402_1005Metric, F.Cu at (43.4, 42.6)
- added C4: 100nF, Capacitor_SMD:C_0603_1608Metric, F.Cu at (20.0, 66.0)
- added C40: 10uF, Capacitor_SMD:C_0805_2012Metric, F.Cu at (24.7, 31.0)
- added C41: 10uF, Capacitor_SMD:C_0805_2012Metric, F.Cu at (24.7, 34.0)
- added C42: 10uF, Capacitor_SMD:C_0805_2012Metric, F.Cu at (24.7, 37.1)
- added C43: 22uF, Capacitor_SMD:C_0805_2012Metric, F.Cu at (24.7, 40.1)
- added C44: 33pF, Capacitor_SMD:C_0402_1005Metric, F.Cu at (43.4, 44.5)
- added C45: 10uF, Capacitor_SMD:C_0805_2012Metric, F.Cu at (29.1, 22.0)
- added C46: 1.8nF, Capacitor_SMD:C_0402_1005Metric, F.Cu at (43.4, 46.5)
- added C47: 4.7uF, Capacitor_SMD:C_0402_1005Metric, F.Cu at (43.4, 48.5)
- added C48: 0.1uF, Capacitor_SMD:C_0402_1005Metric, F.Cu at (43.4, 50.4)
- added C49: 4.7uF, Capacitor_SMD:C_0402_1005Metric, F.Cu at (43.4, 52.4)
- added C5: 0.1uF, Capacitor_SMD:C_0402_1005Metric, F.Cu at (37.6, 44.5)
- added C50: 470nF, Capacitor_SMD:C_0603_1608Metric, F.Cu at (20.0, 73.6)
- added C51: 100nF, Capacitor_SMD:C_0603_1608Metric, F.Cu at (20.0, 76.1)
- added C52: 0.1uF, Capacitor_SMD:C_0402_1005Metric, F.Cu at (43.4, 54.4)
- added C53: 33nF, Capacitor_SMD:C_0603_1608Metric, F.Cu at (24.0, 61.0)
- added C54: 100nF, Capacitor_SMD:C_0603_1608Metric, F.Cu at (24.0, 63.5)
- added C55: 4.7uF, Capacitor_SMD:C_0402_1005Metric, F.Cu at (43.4, 56.3)
- added C56: 100nF, Capacitor_SMD:C_0603_1608Metric, F.Cu at (24.0, 66.0)
- added C57: 33nF, Capacitor_SMD:C_0603_1608Metric, F.Cu at (24.0, 68.6)
- added C58: 10nF, Capacitor_SMD:C_0402_1005Metric, F.Cu at (43.4, 58.3)
- added C59: 1nF, Capacitor_SMD:C_0402_1005Metric, F.Cu at (46.2, 42.6)
- added C6: 10uF, Capacitor_SMD:C_0402_1005Metric, F.Cu at (37.6, 46.5)
- added C60: 680pF, Capacitor_SMD:C_0603_1608Metric, F.Cu at (24.0, 71.1)
- added C61: 15pF, Capacitor_SMD:C_0402_1005Metric, F.Cu at (46.2, 44.5)
- added C62: 330pF, Capacitor_SMD:C_0402_1005Metric, F.Cu at (46.2, 46.5)
- added C63: 330pF, Capacitor_SMD:C_0402_1005Metric, F.Cu at (46.2, 48.5)
- added C64: 47nF, Capacitor_SMD:C_0603_1608Metric, F.Cu at (24.0, 73.6)
- added C65: 47nF, Capacitor_SMD:C_0603_1608Metric, F.Cu at (24.0, 76.1)
- added C66: 1nF, Capacitor_SMD:C_0402_1005Metric, F.Cu at (46.2, 50.4)
- added C67: 1uF, Capacitor_SMD:C_0402_1005Metric, F.Cu at (46.2, 52.4)
- added C68: 10uF, Capacitor_SMD:C_0805_2012Metric, F.Cu at (29.1, 25.0)
- added C69: 0.1uF, Capacitor_SMD:C_0402_1005Metric, F.Cu at (46.2, 54.4)
- added C7: 0.1uF, Capacitor_SMD:C_0402_1005Metric, F.Cu at (37.6, 48.5)
- added C70: 1uF, Capacitor_SMD:C_0402_1005Metric, F.Cu at (46.2, 56.3)
- added C71: 10uF, Capacitor_SMD:C_0805_2012Metric, F.Cu at (29.1, 28.0)
- added C72: 0.1uF, Capacitor_SMD:C_0402_1005Metric, F.Cu at (46.2, 58.3)
- added C73: 470nF, Capacitor_SMD:C_0603_1608Metric, F.Cu at (28.0, 61.0)
- added C74: 0.1uF, Capacitor_SMD:C_0402_1005Metric, F.Cu at (49.1, 42.6)
- added C75: 0.1uF, Capacitor_SMD:C_0402_1005Metric, F.Cu at (49.1, 44.5)
- added C76: 10uF, Capacitor_SMD:C_0805_2012Metric, F.Cu at (29.1, 31.0)
- added C77: 22uF, Capacitor_SMD:C_0805_2012Metric, F.Cu at (29.1, 34.0)
- added C78: 10uF, Capacitor_SMD:C_0805_2012Metric, F.Cu at (29.1, 37.1)
- added C79: 22uF, Capacitor_SMD:C_0805_2012Metric, F.Cu at (29.1, 40.1)
- added C8: 100nF, Capacitor_SMD:C_0603_1608Metric, F.Cu at (20.0, 68.6)
- added C80: 10uF, Capacitor_SMD:C_0805_2012Metric, F.Cu at (33.6, 22.0)
- added C81: 330pF, Capacitor_SMD:C_0402_1005Metric, F.Cu at (49.1, 46.5)
- added C82: 100uF, footprints:CAP-SMD_L7.3-W6.1_TCN4227M025R0100, F.Cu at (40.6, 80.9)
- added C83: 10uF, Capacitor_SMD:C_0805_2012Metric, F.Cu at (33.6, 25.0)
- added C84: 0.1uF, Capacitor_SMD:C_0402_1005Metric, F.Cu at (49.1, 48.5)
- added C85: 0.1uF, Capacitor_SMD:C_0402_1005Metric, F.Cu at (49.1, 50.4)
- added C86: 10uF, Capacitor_SMD:C_0805_2012Metric, F.Cu at (33.6, 28.0)
- added C87: 0.1uF, Capacitor_SMD:C_0402_1005Metric, F.Cu at (49.1, 52.4)
- added C88: 3.3nF, Capacitor_SMD:C_0402_1005Metric, F.Cu at (49.1, 54.4)
- added C9: 22uF, Capacitor_SMD:C_0805_2012Metric, F.Cu at (20.2, 22.0)
- added D1: 30V, PCM_JLCPCB:D_SOT-23, F.Cu at (69.4, 33.5)
- added D10: H5VU25U, PCM_JLCPCB:DFN2510-10_L2.5-W1.0-P0.50-BL, F.Cu at (57.6, 32.8)
- added D11: H5VU25U, PCM_JLCPCB:DFN2510-10_L2.5-W1.0-P0.50-BL, F.Cu at (57.6, 35.6)
- added D2: H5VU25U, PCM_JLCPCB:DFN2510-10_L2.5-W1.0-P0.50-BL, F.Cu at (57.6, 27.1)
- added D3: H5VU25U, PCM_JLCPCB:DFN2510-10_L2.5-W1.0-P0.50-BL, F.Cu at (57.6, 30.0)
- added D4: 30V, PCM_JLCPCB:D_SOT-23, F.Cu at (69.4, 38.1)
- added D5: LED, LED_SMD:LED_0603_1608Metric, F.Cu at (72.5, 61.0)
- added D6: LED, LED_SMD:LED_0603_1608Metric, F.Cu at (72.5, 63.6)
- added D7: LED, LED_SMD:LED_0603_1608Metric, F.Cu at (72.5, 66.2)
- added D8: LED, LED_SMD:LED_0603_1608Metric, F.Cu at (72.5, 68.8)
- added D9: LED, LED_SMD:LED_0603_1608Metric, F.Cu at (72.5, 71.3)
- added FB1: 120, Inductor_SMD:L_0603_1608Metric, F.Cu at (28.0, 63.5)
- added H1: nSWDIO, TestPoint:TestPoint_THTPad_D2.5mm_Drill1.2mm, F.Cu at (20.3, 43.8)
- added H10: oSDA, TestPoint:TestPoint_THTPad_D2.5mm_Drill1.2mm, F.Cu at (29.4, 48.4)
- added H11: oSCL, TestPoint:TestPoint_THTPad_D2.5mm_Drill1.2mm, F.Cu at (29.4, 52.9)
- added H12: oIRQ, TestPoint:TestPoint_THTPad_D2.5mm_Drill1.2mm, F.Cu at (29.4, 57.5)
- added H13: eSDA, TestPoint:TestPoint_THTPad_D2.5mm_Drill1.2mm, F.Cu at (33.9, 43.8)
- added H14: iCHG, TestPoint:TestPoint_Pad_D2.5mm, F.Cu at (33.9, 48.4)
- added H15: eSCL, TestPoint:TestPoint_THTPad_D2.5mm_Drill1.2mm, F.Cu at (33.9, 52.9)
- added H16: GND, TestPoint:TestPoint_THTPad_2.5x2.5mm_Drill1.2mm, F.Cu at (33.9, 57.5)
- added H2: cSDA, TestPoint:TestPoint_THTPad_D2.5mm_Drill1.2mm, F.Cu at (20.3, 48.4)
- added H3: cSCL, TestPoint:TestPoint_THTPad_D2.5mm_Drill1.2mm, F.Cu at (20.3, 52.9)
- added H4: nRST, TestPoint:TestPoint_THTPad_D2.5mm_Drill1.2mm, F.Cu at (20.3, 57.5)
- added H5: nSWDCLK, TestPoint:TestPoint_THTPad_D2.5mm_Drill1.2mm, F.Cu at (24.8, 43.8)
- added H6: bSMBC, TestPoint:TestPoint_THTPad_D2.5mm_Drill1.2mm, F.Cu at (24.8, 48.4)
- added H7: bSMBD, TestPoint:TestPoint_THTPad_D2.5mm_Drill1.2mm, F.Cu at (24.8, 52.9)
- added H8: FUSE, TestPoint:TestPoint_Pad_D2.5mm, F.Cu at (24.8, 57.5)
- added H9: 3V3, TestPoint:TestPoint_THTPad_D2.5mm_Drill1.2mm, F.Cu at (29.4, 43.8)
- added J1: USB_C_Receptacle_USB2.0_16P, footprints:USB-C-SMD_TYPE-C16PIN, F.Cu at (67.1, 95.3)
- added J2: Battery_Connector, footprints:BMS_4S_PAD, F.Cu at (19.9, 79.2)
- added J3: USB_C_Receptacle_USB2.0_16P, footprints:USB-C-SMD_TYPE-C16PIN, F.Cu at (67.2, 126.3)
- added L1: 4.7uH, footprints:IND-SMD_L7.0-W6.6, F.Cu at (65.8, 63.6)
- added L2: 3.5nH, Inductor_SMD:L_0201_0603Metric, F.Cu at (46.0, 35.4)
- added L3: 2.7nH, Inductor_SMD:L_0201_0603Metric, F.Cu at (46.0, 37.2)
- added L4: 3.5nH, Inductor_SMD:L_0201_0603Metric, F.Cu at (46.0, 38.9)
- added L5: 2.2uH, footprints:IND-SMD_L7.1-W6.6, F.Cu at (40.3, 29.7)
- added L6: 4.7uH, footprints:IND-SMD_L7.0-W6.6, F.Cu at (65.8, 71.5)
- added Q1: Q_NMOS, footprints:QNM30N20AJ-PDFN-8L_L3.3-W3.3-P0.65-BL_XINFEIHONG_FH1404G6, F.Cu at (38.0, 22.9)
- added Q2: Q_PMOS, footprints:ZC015P2G-POWERTDFN-8_L3.1-W3.1-P0.65-LS3.3-BL, F.Cu at (69.2, 28.2)
- added Q3: Q_NMOS, footprints:QNM30N20AJ-PDFN-8L_L3.3-W3.3-P0.65-BL_XINFEIHONG_FH1404G6, F.Cu at (42.5, 22.9)
- added Q4: Q_NMOS, footprints:QNM30N20AJ-PDFN-8L_L3.3-W3.3-P0.65-BL_XINFEIHONG_FH1404G6, F.Cu at (47.0, 22.9)
- added Q5: Q_NMOS, footprints:QNM30N20AJ-PDFN-8L_L3.3-W3.3-P0.65-BL_XINFEIHONG_FH1404G6, F.Cu at (51.5, 22.9)
- added Q6: Q_NMOS, footprints:QNM30N20AJ-PDFN-8L_L3.3-W3.3-P0.65-BL_XINFEIHONG_FH1404G6, F.Cu at (56.0, 22.9)
- added Q7: Q_NMOS, footprints:QNM30N20AJ-PDFN-8L_L3.3-W3.3-P0.65-BL_XINFEIHONG_FH1404G6, F.Cu at (60.5, 22.9)
- added Q8: Q_NMOS, footprints:QNM30N20AJ-PDFN-8L_L3.3-W3.3-P0.65-BL_XINFEIHONG_FH1404G6, F.Cu at (65.0, 22.9)
- added Q9: Q_PMOS, footprints:ZC015P2G-POWERTDFN-8_L3.1-W3.1-P0.65-LS3.3-BL, F.Cu at (73.8, 28.2)
- added R1: DNP, Resistor_SMD:R_0603_1608Metric, F.Cu at (28.0, 66.0)
- added R10: 200, Resistor_SMD:R_0402_1005Metric_Pad0.72x0.64mm_HandSolder, F.Cu at (77.4, 38.5)
- added R11: 200, Resistor_SMD:R_0402_1005Metric_Pad0.72x0.64mm_HandSolder, F.Cu at (77.4, 40.5)
- added R12: 100, Resistor_SMD:R_0402_1005Metric, F.Cu at (37.7, 64.3)
- added R13: 100, Resistor_SMD:R_0402_1005Metric, F.Cu at (37.7, 66.3)
- added R14: 10M, Resistor_SMD:R_0402_1005Metric, F.Cu at (37.7, 68.3)
- added R15: 300, Resistor_SMD:R_1206_3216Metric, F.Cu at (77.2, 43.2)
- added R16: 5.1k, Resistor_SMD:R_0402_1005Metric, F.Cu at (37.7, 70.2)
- added R17: 5.1k, Resistor_SMD:R_0402_1005Metric, F.Cu at (37.7, 72.2)
- added R18: 10M, Resistor_SMD:R_0402_1005Metric, F.Cu at (37.7, 74.2)
- added R19: 100, Resistor_SMD:R_0402_1005Metric, F.Cu at (37.7, 76.2)
- added R2: 0, Resistor_SMD:R_0603_1608Metric, F.Cu at (28.0, 68.6)
- added R20: 100, Resistor_SMD:R_0402_1005Metric, F.Cu at (40.6, 60.3)
- added R21: 100, Resistor_SMD:R_0402_1005Metric, F.Cu at (40.6, 62.3)
- added R22: 100, Resistor_SMD:R_0402_1005Metric, F.Cu at (40.6, 64.3)
- added R23: 100, Resistor_SMD:R_0402_1005Metric, F.Cu at (40.6, 66.3)
- added R24: 5.1k, Resistor_SMD:R_0402_1005Metric, F.Cu at (40.6, 68.3)
- added R25: 10M, Resistor_SMD:R_0402_1005Metric, F.Cu at (40.6, 70.2)
- added R26: 10k, Resistor_SMD:R_0805_2012Metric, F.Cu at (63.4, 48.9)
- added R27: 10k, Resistor_SMD:R_0805_2012Metric, F.Cu at (63.4, 51.9)
- added R28: 100, Resistor_SMD:R_0402_1005Metric, F.Cu at (40.6, 72.2)
- added R29: 1m, Resistor_SMD:R_1206_3216Metric, F.Cu at (77.2, 46.5)
- added R3: 10k, Resistor_SMD:R_0805_2012Metric, F.Cu at (63.4, 43.0)
- added R30: 10k, Resistor_SMD:R_0805_2012Metric, F.Cu at (63.4, 54.8)
- added R31: 100, Resistor_SMD:R_0402_1005Metric, F.Cu at (40.6, 74.2)
- added R32: 5.6k, Resistor_SMD:R_0402_1005Metric, F.Cu at (40.6, 76.2)
- added R33: 10, Resistor_SMD:R_0402_1005Metric, F.Cu at (43.5, 60.3)
- added R34: 10k, Resistor_SMD:R_0805_2012Metric, F.Cu at (67.8, 43.0)
- added R35: 10k, Resistor_SMD:R_0805_2012Metric, F.Cu at (67.8, 46.0)
- added R36: 220k, Resistor_SMD:R_0402_1005Metric, F.Cu at (43.5, 62.3)
- added R37: 22k, Resistor_SMD:R_0402_1005Metric, F.Cu at (43.5, 64.3)
- added R38: 4.7k, Resistor_SMD:R_0402_1005Metric, F.Cu at (43.5, 66.3)
- added R39: 40.2k, Resistor_SMD:R_0603_1608Metric, F.Cu at (28.0, 76.1)
- added R4: 220k, Resistor_SMD:R_0402_1005Metric, F.Cu at (37.7, 60.3)
- added R40: 4.7k, Resistor_SMD:R_0402_1005Metric, F.Cu at (43.5, 68.3)
- added R41: 1, Resistor_SMD:R_0402_1005Metric, F.Cu at (43.5, 70.2)
- added R42: 4.7k, Resistor_SMD:R_0402_1005Metric, F.Cu at (43.5, 72.2)
- added R43: 4.7, Resistor_SMD:R_0603_1608Metric, F.Cu at (32.0, 61.0)
- added R44: 10m, Resistor_SMD:R_1206_3216Metric, F.Cu at (77.2, 49.8)
- added R45: 4.7, Resistor_SMD:R_0603_1608Metric, F.Cu at (32.0, 63.5)
- added R46: 4.7k, Resistor_SMD:R_0402_1005Metric, F.Cu at (43.5, 74.2)
- added R47: 10k, Resistor_SMD:R_0805_2012Metric, F.Cu at (67.8, 48.9)
- added R48: 10k, Resistor_SMD:R_0805_2012Metric, F.Cu at (67.8, 51.9)
- added R49: 220k, Resistor_SMD:R_0402_1005Metric, F.Cu at (43.5, 76.2)
- added R5: 160k, Resistor_SMD:R_0603_1608Metric, F.Cu at (28.0, 71.1)
- added R50: 2.2, Resistor_SMD:R_0805_2012Metric, F.Cu at (67.8, 54.8)
- added R51: 10, Resistor_SMD:R_0402_1005Metric, F.Cu at (46.4, 60.3)
- added R52: 2.2, Resistor_SMD:R_0805_2012Metric, F.Cu at (72.2, 43.0)
- added R53: 390k, Resistor_SMD:R_0603_1608Metric, F.Cu at (32.0, 66.0)
- added R54: 220k, Resistor_SMD:R_0402_1005Metric, F.Cu at (46.4, 62.3)
- added R55: 10, Resistor_SMD:R_0402_1005Metric, F.Cu at (46.4, 64.3)
- added R56: 10m, Resistor_SMD:R_1206_3216Metric, F.Cu at (77.2, 53.2)
- added R57: 0, Resistor_SMD:R_0603_1608Metric, F.Cu at (32.0, 68.6)
- added R58: 10, Resistor_SMD:R_0402_1005Metric, F.Cu at (46.4, 66.3)
- added R59: 10, Resistor_SMD:R_0402_1005Metric, F.Cu at (46.4, 68.3)
- added R60: 10m, Resistor_SMD:R_1206_3216Metric, F.Cu at (77.2, 56.5)
- added R61: 4.7k, Resistor_SMD:R_0402_1005Metric, F.Cu at (46.4, 70.2)
- added R62: 4.7k, Resistor_SMD:R_0402_1005Metric, F.Cu at (46.4, 72.2)
- added R63: 137k, Resistor_SMD:R_0603_1608Metric, F.Cu at (32.0, 71.1)
- added R64: 2.2, Resistor_SMD:R_0805_2012Metric, F.Cu at (72.2, 46.0)
- added R65: 2.2, Resistor_SMD:R_0805_2012Metric, F.Cu at (72.2, 48.9)
- added R66: 40.2k, Resistor_SMD:R_0603_1608Metric, F.Cu at (32.0, 73.6)
- added R7: 220k, Resistor_SMD:R_0402_1005Metric, F.Cu at (37.7, 62.3)
- added R8: 10k, Resistor_SMD:R_0805_2012Metric, F.Cu at (63.4, 46.0)
- added R9: 1k, Resistor_SMD:R_0603_1608Metric, F.Cu at (28.0, 73.6)
- added SW1: SW_Push, Button_Switch_THT:SW_PUSH_6mm, F.Cu at (52.6, 61.7)
- added SW2: SW_Push, Button_Switch_THT:SW_PUSH_6mm, F.Cu at (52.6, 70.3)
- added SW3: SW_Push, Connector_Wire:SolderWire-0.127sqmm_1x02_P3.7mm_D0.48mm_OD1mm, F.Cu at (61.4, 27.7)
- added TH1: 10k, Connector_Wire:SolderWire-0.127sqmm_1x02_P3.7mm_D0.48mm_OD1mm, F.Cu at (61.4, 31.4)
- added U1: nRF54L10-QFXX, Package_DFN_QFN:QFN-48-1EP_6x6mm_P0.4mm_EP4.6x4.6mm_ThermalVias, F.Cu at (55.0, 80.9)
- added U2: TPS25730DREFR, footprints:REF0038A-MFG, F.Cu at (51.7, 35.5)
- added U3: BQ4050RSMR, footprints:VQFN-32_L4.0-W4.0-P0.40-TL-EP1.4, F.Cu at (39.0, 36.6)
- added U4: BQ25713RSNR, footprints:RSN32_TEX, F.Cu at (75.1, 34.3)
- added U5: TPS25762DQRQLRQ1, footprints:RQL0029A-MFG, F.Cu at (51.7, 29.3)
- added U6: AT24C256C-SSHL-T, footprints:SOIC-8_L4.9-W3.9-P1.27-LS6.0-BL, F.Cu at (63.0, 37.4)
- added X1: 32MHz, footprints:CRYSTAL-SMD_4P-L2.0-W1.6-BL-A, F.Cu at (73.9, 39.1)
Other:
- board outline added: 74 x 51.5 mm

Commit message: a
Parts:
- moved J3 70.0 mm to (56.9, 57.1), turned to 0 degrees
- moved J1 48.4 mm to (56.9, 48.0), turned to 0 degrees
- moved C1 3.16 mm to (21.0, 64.0)
- moved C53 3.16 mm to (25.0, 64.0)
- moved C73 3.16 mm to (29.0, 64.0)
- moved R43 3.16 mm to (33.0, 64.0)
- moved AE1 3.16 mm to (65.9, 84.6)
- moved C10 3.16 mm to (21.2, 28.0)
- moved C11 3.16 mm to (21.2, 31.0)
- moved C13 3.16 mm to (47.0, 29.7)
- moved C14 3.16 mm to (21.2, 37.0)
- moved C15 3.16 mm to (38.6, 53.4)
- moved C16 3.16 mm to (47.0, 31.4)
- moved C17 3.16 mm to (47.0, 33.2)
- moved C18 3.16 mm to (38.6, 55.4)
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
Commit message: rean
Parts:
- removed AE1: Antenna, RF_Antenna:Texas_SWRA117D_2.4GHz_Right
- removed C1, C2, C4, C51, C54, C56, C8: 100nF, Capacitor_SMD:C_0603_1608Metric
- removed C10, C19, C36, C38, C40, C41, C42, C45, C68, C71, C76, C78, C80, C83, C86: 10uF, Capacitor_SMD:C_0805_2012Metric
- removed C11, C12, C21, C26: 2.2uF, Capacitor_SMD:C_0805_2012Metric
- removed C13, C22: 2pF, Capacitor_SMD:C_0201_0603Metric
- removed C14, C43, C77, C79, C9: 22uF, Capacitor_SMD:C_0805_2012Metric
- removed C15, C18, C6: 10uF, Capacitor_SMD:C_0402_1005Metric
- removed C16: 10nF, Capacitor_SMD:C_0201_0603Metric
- removed C17: 1.5pF, Capacitor_SMD:C_0201_0603Metric
- removed C20, C47, C49, C55: 4.7uF, Capacitor_SMD:C_0402_1005Metric
- removed C23: 0.3pF, Capacitor_SMD:C_0201_0603Metric
- removed C24, C25, C62, C63, C81: 330pF, Capacitor_SMD:C_0402_1005Metric
- removed C27, C28, C29, C3, C30, C31, C32, C33, C34, C35, C39, C48, C5, C52, C69, C7, C72, C74, C75, C84, C85, C87: 0.1uF, Capacitor_SMD:C_0402_1005Metric
- removed C37, C50, C73: 470nF, Capacitor_SMD:C_0603_1608Metric
- removed C44: 33pF, Capacitor_SMD:C_0402_1005Metric
- removed C46: 1.8nF, Capacitor_SMD:C_0402_1005Metric
- removed C53, C57: 33nF, Capacitor_SMD:C_0603_1608Metric
- removed C58: 10nF, Capacitor_SMD:C_0402_1005Metric
- removed C59, C66: 1nF, Capacitor_SMD:C_0402_1005Metric
- removed C60: 680pF, Capacitor_SMD:C_0603_1608Metric
- removed C61: 15pF, Capacitor_SMD:C_0402_1005Metric
- removed C64, C65: 47nF, Capacitor_SMD:C_0603_1608Metric
- removed C67, C70: 1uF, Capacitor_SMD:C_0402_1005Metric
- removed C82: 100uF, footprints:CAP-SMD_L7.3-W6.1_TCN4227M025R0100
- removed C88: 3.3nF, Capacitor_SMD:C_0402_1005Metric
- removed D1, D4: 30V, PCM_JLCPCB:D_SOT-23
- removed D10, D11, D2, D3: H5VU25U, PCM_JLCPCB:DFN2510-10_L2.5-W1.0-P0.50-BL
- removed D5, D6, D7, D8, D9: LED, LED_SMD:LED_0603_1608Metric
- removed FB1: 120, Inductor_SMD:L_0603_1608Metric
- removed H1: nSWDIO, TestPoint:TestPoint_THTPad_D2.5mm_Drill1.2mm
- removed H10: oSDA, TestPoint:TestPoint_THTPad_D2.5mm_Drill1.2mm
- removed H11: oSCL, TestPoint:TestPoint_THTPad_D2.5mm_Drill1.2mm
- removed H12: oIRQ, TestPoint:TestPoint_THTPad_D2.5mm_Drill1.2mm
- removed H13: eSDA, TestPoint:TestPoint_THTPad_D2.5mm_Drill1.2mm
- removed H14: iCHG, TestPoint:TestPoint_Pad_D2.5mm
- removed H15: eSCL, TestPoint:TestPoint_THTPad_D2.5mm_Drill1.2mm
- removed H16: GND, TestPoint:TestPoint_THTPad_2.5x2.5mm_Drill1.2mm
- removed H2: cSDA, TestPoint:TestPoint_THTPad_D2.5mm_Drill1.2mm
- removed H3: cSCL, TestPoint:TestPoint_THTPad_D2.5mm_Drill1.2mm
- removed H4: nRST, TestPoint:TestPoint_THTPad_D2.5mm_Drill1.2mm
- removed H5: nSWDCLK, TestPoint:TestPoint_THTPad_D2.5mm_Drill1.2mm
- removed H6: bSMBC, TestPoint:TestPoint_THTPad_D2.5mm_Drill1.2mm
- removed H7: bSMBD, TestPoint:TestPoint_THTPad_D2.5mm_Drill1.2mm
- removed H8: FUSE, TestPoint:TestPoint_Pad_D2.5mm
- removed H9: 3V3, TestPoint:TestPoint_THTPad_D2.5mm_Drill1.2mm
- removed J1, J3: USB_C_Receptacle_USB2.0_16P, footprints:USB-C-SMD_TYPE-C16PIN
- removed J2: Battery_Connector, footprints:BMS_4S_PAD
- removed L1, L6: 4.7uH, footprints:IND-SMD_L7.0-W6.6
- removed L2, L4: 3.5nH, Inductor_SMD:L_0201_0603Metric
- removed L3: 2.7nH, Inductor_SMD:L_0201_0603Metric
- removed L5: 2.2uH, footprints:IND-SMD_L7.1-W6.6
- removed Q1, Q3, Q4, Q5, Q6, Q7, Q8: Q_NMOS, footprints:QNM30N20AJ-PDFN-8L_L3.3-W3.3-P0.65-BL_XINFEIHONG_FH1404G6
- removed Q2, Q9: Q_PMOS, footprints:ZC015P2G-POWERTDFN-8_L3.1-W3.1-P0.65-LS3.3-BL
- removed R1: DNP, Resistor_SMD:R_0603_1608Metric
- removed R10, R11: 200, Resistor_SMD:R_0402_1005Metric_Pad0.72x0.64mm_HandSolder
- removed R12, R13, R19, R20, R21, R22, R23, R28, R31: 100, Resistor_SMD:R_0402_1005Metric
- removed R14, R18, R25: 10M, Resistor_SMD:R_0402_1005Metric
- removed R15: 300, Resistor_SMD:R_1206_3216Metric
- removed R16, R17, R24: 5.1k, Resistor_SMD:R_0402_1005Metric
- removed R2, R57: 0, Resistor_SMD:R_0603_1608Metric
- removed R26, R27, R3, R30, R34, R35, R47, R48, R8: 10k, Resistor_SMD:R_0805_2012Metric
- removed R29: 1m, Resistor_SMD:R_1206_3216Metric
- removed R32: 5.6k, Resistor_SMD:R_0402_1005Metric
- removed R33, R51, R55, R58, R59: 10, Resistor_SMD:R_0402_1005Metric
- removed R36, R4, R49, R54, R7: 220k, Resistor_SMD:R_0402_1005Metric
- removed R37: 22k, Resistor_SMD:R_0402_1005Metric
- removed R38, R40, R42, R46, R61, R62: 4.7k, Resistor_SMD:R_0402_1005Metric
- removed R39, R66: 40.2k, Resistor_SMD:R_0603_1608Metric
- removed R41: 1, Resistor_SMD:R_0402_1005Metric
- removed R43, R45: 4.7, Resistor_SMD:R_0603_1608Metric
- removed R44, R56, R60: 10m, Resistor_SMD:R_1206_3216Metric
- removed R5: 160k, Resistor_SMD:R_0603_1608Metric
- removed R50, R52, R64, R65: 2.2, Resistor_SMD:R_0805_2012Metric
- removed R53: 390k, Resistor_SMD:R_0603_1608Metric
- removed R63: 137k, Resistor_SMD:R_0603_1608Metric
- removed R9: 1k, Resistor_SMD:R_0603_1608Metric
- removed SW1, SW2: SW_Push, Button_Switch_THT:SW_PUSH_6mm
- removed SW3: SW_Push, Connector_Wire:SolderWire-0.127sqmm_1x02_P3.7mm_D0.48mm_OD1mm
- removed TH1: 10k, Connector_Wire:SolderWire-0.127sqmm_1x02_P3.7mm_D0.48mm_OD1mm
- removed U1: nRF54L10-QFXX, Package_DFN_QFN:QFN-48-1EP_6x6mm_P0.4mm_EP4.6x4.6mm_ThermalVias
- removed U2: TPS25730DREFR, footprints:REF0038A-MFG
- removed U3: BQ4050RSMR, footprints:VQFN-32_L4.0-W4.0-P0.40-TL-EP1.4
- removed U4: BQ25713RSNR, footprints:RSN32_TEX
- removed U5: TPS25762DQRQLRQ1, footprints:RQL0029A-MFG
- removed U6: AT24C256C-SSHL-T, footprints:SOIC-8_L4.9-W3.9-P1.27-LS6.0-BL
- removed X1: 32MHz, footprints:CRYSTAL-SMD_4P-L2.0-W1.6-BL-A
Other:
- copper layers 2 -> 4
