File: pcb/FindMyCharger.kicad_pcb (KiCad board)
At the start: 4 copper layers, 74 x 51.5 mm, 0 parts

Commit message: dum
Parts:
- added AE1: Antenna, RF_Antenna:Texas_SWRA117D_2.4GHz_Right, F.Cu at (159.8, 135.2)
- added C1: 10uF, Capacitor_SMD:C_0402_1005Metric, F.Cu at (122.0, 92.0)
- added C10: 10uF, Capacitor_SMD:C_0805_2012Metric, F.Cu at (72.1, 156.0)
- added C11: 0.1uF, Capacitor_SMD:C_0402_1005Metric, F.Cu at (103.0, 99.9)
- added C12: 10uF, Capacitor_SMD:C_0805_2012Metric, F.Cu at (98.0, 95.0)
- added C13: 22uF, Capacitor_SMD:C_0805_2012Metric, F.Cu at (100.0, 95.0)
- added C14: 22uF, Capacitor_SMD:C_0805_2012Metric, F.Cu at (102.0, 95.0)
- added C15: 10uF, Capacitor_SMD:C_0805_2012Metric, F.Cu at (111.0, 103.0)
- added C16: 10uF, Capacitor_SMD:C_0805_2012Metric, F.Cu at (134.6, 119.0)
- added C17: 10uF, Capacitor_SMD:C_0805_2012Metric, F.Cu at (134.6, 122.0)
- added C18: 10uF, Capacitor_SMD:C_0805_2012Metric, F.Cu at (134.6, 125.0)
- added C19: 10uF, Capacitor_SMD:C_0805_2012Metric, F.Cu at (139.0, 119.2)
- added C2: 0.1uF, Capacitor_SMD:C_0402_1005Metric, F.Cu at (98.0, 99.0)
- added C20: 10uF, Capacitor_SMD:C_0805_2012Metric, F.Cu at (139.0, 122.3)
- added C21: 10uF, Capacitor_SMD:C_0805_2012Metric, F.Cu at (139.0, 125.3)
- added C22: 10nF, Capacitor_SMD:C_0402_1005Metric, F.Cu at (48.2, 131.7)
- added C23: 1nF, Capacitor_SMD:C_0402_1005Metric, F.Cu at (48.2, 133.6)
- added C24: 47nF, Capacitor_SMD:C_0603_1608Metric, F.Cu at (114.2, 107.5)
- added C25: 47nF, Capacitor_SMD:C_0603_1608Metric, F.Cu at (114.2, 110.0)
- added C26: 0.1uF, Capacitor_SMD:C_0402_1005Metric, F.Cu at (48.2, 135.6)
- added C27: 330pF, Capacitor_SMD:C_0402_1005Metric, F.Cu at (98.0, 101.0)
- added C28: 330pF, Capacitor_SMD:C_0402_1005Metric, F.Cu at (98.0, 103.0)
- added C29: 1uF, Capacitor_SMD:C_0402_1005Metric, F.Cu at (51.0, 123.8)
- added C3: 0.1uF, Capacitor_SMD:C_0402_1005Metric, F.Cu at (98.0, 105.0)
- added C30: 10uF, Capacitor_SMD:C_0402_1005Metric, F.Cu at (122.5, 94.5)
- added C31: 33nF, Capacitor_SMD:C_0603_1608Metric, F.Cu at (114.2, 112.5)
- added C32: 33nF, Capacitor_SMD:C_0603_1608Metric, F.Cu at (118.0, 107.5)
- added C33: 4.7uF, Capacitor_SMD:C_0402_1005Metric, F.Cu at (122.5, 96.5)
- added C34: 470nF, Capacitor_SMD:C_0603_1608Metric, F.Cu at (118.0, 110.0)
- added C35: 1uF, Capacitor_SMD:C_0402_1005Metric, F.Cu at (51.0, 129.7)
- added C36: 330pF, Capacitor_SMD:C_0402_1005Metric, F.Cu at (51.0, 131.7)
- added C37: 0.1uF, Capacitor_SMD:C_0402_1005Metric, F.Cu at (140.0, 128.3)
- added C38: 0.1uF, Capacitor_SMD:C_0402_1005Metric, F.Cu at (140.0, 130.2)
- added C39: 33pF, Capacitor_SMD:C_0402_1005Metric, F.Cu at (51.0, 137.6)
- added C4: 10uF, Capacitor_SMD:C_0805_2012Metric, F.Cu at (72.1, 138.0)
- added C40: 15pF, Capacitor_SMD:C_0402_1005Metric, F.Cu at (51.0, 139.5)
- added C41: 1.8nF, Capacitor_SMD:C_0402_1005Metric, F.Cu at (53.9, 123.8)
- added C42: 680pF, Capacitor_SMD:C_0603_1608Metric, F.Cu at (118.0, 112.5)
- added C43: 100nF, Capacitor_SMD:C_0603_1608Metric, F.Cu at (154.8, 127.8)
- added C44: 100nF, Capacitor_SMD:C_0603_1608Metric, F.Cu at (158.3, 123.8)
- added C45: 100nF, Capacitor_SMD:C_0603_1608Metric, F.Cu at (158.3, 126.3)
- added C46: 10uF, Capacitor_SMD:C_0402_1005Metric, F.Cu at (154.8, 124.8)
- added C47: 100nF, Capacitor_SMD:C_0603_1608Metric, F.Cu at (158.3, 128.8)
- added C48: 0.1uF, Capacitor_SMD:C_0402_1005Metric, F.Cu at (53.9, 127.7)
- added C49: 0.1uF, Capacitor_SMD:C_0402_1005Metric, F.Cu at (53.9, 129.7)
- added C5: 10uF, Capacitor_SMD:C_0805_2012Metric, F.Cu at (72.1, 141.0)
- added C50: 1nF, Capacitor_SMD:C_0402_1005Metric, F.Cu at (53.9, 131.7)
- added C51: 3.3nF, Capacitor_SMD:C_0402_1005Metric, F.Cu at (53.9, 133.6)
- added C52: 0.1uF, Capacitor_SMD:C_0402_1005Metric, F.Cu at (53.9, 135.6)
- added C53: 0.1uF, Capacitor_SMD:C_0402_1005Metric, F.Cu at (53.9, 137.6)
- added C54: 2.2uF, Capacitor_SMD:C_0805_2012Metric, F.Cu at (81.0, 147.0)
- added C55: 470nF, Capacitor_SMD:C_0603_1608Metric, F.Cu at (124.0, 138.0)
- added C56: 0.1uF, Capacitor_SMD:C_0402_1005Metric, F.Cu at (53.9, 139.5)
- added C57: 0.1uF, Capacitor_SMD:C_0402_1005Metric, F.Cu at (56.8, 123.8)
- added C58: 0.1uF, Capacitor_SMD:C_0402_1005Metric, F.Cu at (142.6, 114.8)
- added C59: 2.2uF, Capacitor_SMD:C_0805_2012Metric, F.Cu at (81.0, 150.0)
- added C6: 10uF, Capacitor_SMD:C_0805_2012Metric, F.Cu at (72.1, 144.0)
- added C60: 10nF, Capacitor_SMD:C_0201_0603Metric, F.Cu at (160.9, 110.5)
- added C61: 2.2uF, Capacitor_SMD:C_0805_2012Metric, F.Cu at (81.0, 153.0)
- added C62: 4.7uF, Capacitor_SMD:C_0402_1005Metric, F.Cu at (130.9, 139.2)
- added C63: 100nF, Capacitor_SMD:C_0603_1608Metric, F.Cu at (128.0, 134.0)
- added C64: 0.1uF, Capacitor_SMD:C_0402_1005Metric, F.Cu at (111.6, 124.5)
- added C65: 0.1uF, Capacitor_SMD:C_0402_1005Metric, F.Cu at (111.6, 126.5)
- added C66: 22uF, Capacitor_SMD:C_0805_2012Metric, F.Cu at (107.6, 128.0)
- added C67: 22uF, Capacitor_SMD:C_0805_2012Metric, F.Cu at (108.0, 123.0)
- added C68: 100uF, footprints:CAP-SMD_L7.3-W6.1_TCN4227M025R0100, F.Cu at (105.5, 135.5)
- added C69: 0.1uF, Capacitor_SMD:C_0402_1005Metric, F.Cu at (99.5, 135.5)
- added C7: 10uF, Capacitor_SMD:C_0805_2012Metric, F.Cu at (72.1, 147.0)
- added C70: 0.1uF, Capacitor_SMD:C_0402_1005Metric, F.Cu at (99.5, 137.5)
- added C71: 0.1uF, Capacitor_SMD:C_0402_1005Metric, F.Cu at (137.0, 110.8)
- added C72: 0.1uF, Capacitor_SMD:C_0402_1005Metric, F.Cu at (137.0, 112.7)
- added C73: 4.7uF, Capacitor_SMD:C_0402_1005Metric, F.Cu at (133.5, 137.5)
- added C74: 100nF, Capacitor_SMD:C_0603_1608Metric, F.Cu at (128.0, 136.5)
- added C75: 1.5pF, Capacitor_SMD:C_0201_0603Metric, F.Cu at (160.9, 112.2)
- added C76: 2pF, Capacitor_SMD:C_0201_0603Metric, F.Cu at (160.9, 114.0)
- added C77: 0.3pF, Capacitor_SMD:C_0201_0603Metric, F.Cu at (160.9, 115.8)
- added C78: 4.7uF, Capacitor_SMD:C_0402_1005Metric, F.Cu at (133.5, 139.5)
- added C79: 100nF, Capacitor_SMD:C_0603_1608Metric, F.Cu at (128.0, 139.0)
- added C8: 10uF, Capacitor_SMD:C_0805_2012Metric, F.Cu at (72.1, 150.0)
- added C80: 2.2uF, Capacitor_SMD:C_0805_2012Metric, F.Cu at (85.5, 141.0)
- added C81: 330pF, Capacitor_SMD:C_0402_1005Metric, F.Cu at (59.6, 127.7)
- added C82: 22uF, Capacitor_SMD:C_0805_2012Metric, F.Cu at (136.8, 129.2)
- added C83: 0.1uF, Capacitor_SMD:C_0402_1005Metric, F.Cu at (131.0, 134.3)
- added C84: 0.1uF, Capacitor_SMD:C_0402_1005Metric, F.Cu at (131.0, 136.2)
- added C85: 2pF, Capacitor_SMD:C_0201_0603Metric, F.Cu at (160.9, 117.5)
- added C86: 470nF, Capacitor_SMD:C_0603_1608Metric, F.Cu at (38.6, 142.2)
- added C87: 0.1uF, Capacitor_SMD:C_0402_1005Metric, F.Cu at (59.6, 133.6)
- added C88: 330pF, Capacitor_SMD:C_0402_1005Metric, F.Cu at (59.6, 135.6)
- added C9: 10uF, Capacitor_SMD:C_0805_2012Metric, F.Cu at (72.1, 153.0)
- added D1: 30V, PCM_JLCPCB:D_SOT-23, F.Cu at (105.0, 94.6)
- added D10: LED, LED_SMD:LED_0603_1608Metric, F.Cu at (92.3, 117.4)
- added D11: LED, LED_SMD:LED_0603_1608Metric, F.Cu at (92.3, 120.0)
- added D2: H5VU25U, PCM_JLCPCB:DFN2510-10_L2.5-W1.0-P0.50-BL, F.Cu at (105.5, 87.6)
- added D3: 30V, PCM_JLCPCB:D_SOT-23, F.Cu at (147.8, 105.2)
- added D4: H5VU25U, PCM_JLCPCB:DFN2510-10_L2.5-W1.0-P0.50-BL, F.Cu at (168.0, 110.9)
- added D5: H5VU25U, PCM_JLCPCB:DFN2510-10_L2.5-W1.0-P0.50-BL, F.Cu at (168.0, 113.7)
- added D6: H5VU25U, PCM_JLCPCB:DFN2510-10_L2.5-W1.0-P0.50-BL, F.Cu at (168.0, 116.6)
- added D7: LED, LED_SMD:LED_0603_1608Metric, F.Cu at (92.3, 112.4)
- added D8: LED, LED_SMD:LED_0603_1608Metric, F.Cu at (92.3, 115.0)
- added D9: LED, LED_SMD:LED_0603_1608Metric, F.Cu at (92.3, 110.0)
- added FB1: 120, Inductor_SMD:L_0603_1608Metric, F.Cu at (157.0, 109.5)
- added H1: cSDA, TestPoint:TestPoint_THTPad_D2.5mm_Drill1.2mm, F.Cu at (166.0, 124.5)
- added H10: FUSE, TestPoint:TestPoint_Pad_D2.5mm, F.Cu at (175.1, 129.1)
- added H11: eSCL, TestPoint:TestPoint_THTPad_D2.5mm_Drill1.2mm, F.Cu at (175.1, 133.6)
- added H12: bSMBD, TestPoint:TestPoint_THTPad_D2.5mm_Drill1.2mm, F.Cu at (175.1, 138.2)
- added H13: nSWDCLK, TestPoint:TestPoint_THTPad_D2.5mm_Drill1.2mm, F.Cu at (179.7, 124.5)
- added H14: eSDA, TestPoint:TestPoint_THTPad_D2.5mm_Drill1.2mm, F.Cu at (179.7, 129.1)
- added H15: GND, TestPoint:TestPoint_THTPad_2.5x2.5mm_Drill1.2mm, F.Cu at (179.7, 133.6)
- added H16: nSWDIO, TestPoint:TestPoint_THTPad_D2.5mm_Drill1.2mm, F.Cu at (179.7, 138.2)
- added H2: cSCL, TestPoint:TestPoint_THTPad_D2.5mm_Drill1.2mm, F.Cu at (166.0, 129.1)
- added H3: iCHG, TestPoint:TestPoint_Pad_D2.5mm, F.Cu at (166.0, 133.6)
- added H4: oIRQ, TestPoint:TestPoint_THTPad_D2.5mm_Drill1.2mm, F.Cu at (166.0, 138.2)
- added H5: oSCL, TestPoint:TestPoint_THTPad_D2.5mm_Drill1.2mm, F.Cu at (170.6, 124.5)
- added H6: oSDA, TestPoint:TestPoint_THTPad_D2.5mm_Drill1.2mm, F.Cu at (170.6, 129.1)
- added H7: 3V3, TestPoint:TestPoint_THTPad_D2.5mm_Drill1.2mm, F.Cu at (170.6, 133.6)
- added H8: bSMBC, TestPoint:TestPoint_THTPad_D2.5mm_Drill1.2mm, F.Cu at (170.6, 138.2)
- added H9: nRST, TestPoint:TestPoint_THTPad_D2.5mm_Drill1.2mm, F.Cu at (175.1, 124.5)
- added J1: USB_C_Receptacle_USB2.0_16P, footprints:USB-C-SMD_TYPE-C16PIN, F.Cu at (94.1, 102.0)
- added J2: USB_C_Receptacle_USB2.0_16P, footprints:USB-C-SMD_TYPE-C16PIN, F.Cu at (94.0, 127.0)
- added J3: Battery_Connector, footprints:BMS_4S_PAD, F.Cu at (146.0, 91.5)
- added L1: 2.2uH, footprints:IND-SMD_L7.1-W6.6, F.Cu at (131.5, 98.5)
- added L2: 4.7uH, footprints:IND-SMD_L7.0-W6.6, F.Cu at (118.0, 146.0)
- added L3: 4.7uH, footprints:IND-SMD_L7.0-W6.6, F.Cu at (161.2, 100.5)
- added L4: 2.7nH, Inductor_SMD:L_0201_0603Metric, F.Cu at (160.9, 119.2)
- added L5: 3.5nH, Inductor_SMD:L_0201_0603Metric, F.Cu at (160.9, 121.0)
- added L6: 3.5nH, Inductor_SMD:L_0201_0603Metric, F.Cu at (160.9, 122.8)
- added Q1: Q_NMOS, footprints:QNM30N20AJ-PDFN-8L_L3.3-W3.3-P0.65-BL_XINFEIHONG_FH1404G6, F.Cu at (110.5, 117.0)
- added Q2: Q_NMOS, footprints:QNM30N20AJ-PDFN-8L_L3.3-W3.3-P0.65-BL_XINFEIHONG_FH1404G6, F.Cu at (115.0, 117.0)
- added Q3: Q_PMOS, footprints:ZC015P2G-POWERTDFN-8_L3.1-W3.1-P0.65-LS3.3-BL, F.Cu at (128.0, 118.8)
- added Q4: Q_NMOS, footprints:QNM30N20AJ-PDFN-8L_L3.3-W3.3-P0.65-BL_XINFEIHONG_FH1404G6, F.Cu at (119.5, 117.0)
- added Q5: Q_NMOS, footprints:QNM30N20AJ-PDFN-8L_L3.3-W3.3-P0.65-BL_XINFEIHONG_FH1404G6, F.Cu at (124.0, 117.0)
- added Q6: Q_PMOS, footprints:ZC015P2G-POWERTDFN-8_L3.1-W3.1-P0.65-LS3.3-BL, F.Cu at (143.1, 105.9)
- added Q7: Q_NMOS, footprints:QNM30N20AJ-PDFN-8L_L3.3-W3.3-P0.65-BL_XINFEIHONG_FH1404G6, F.Cu at (146.0, 110.5)
- added Q8: Q_NMOS, footprints:QNM30N20AJ-PDFN-8L_L3.3-W3.3-P0.65-BL_XINFEIHONG_FH1404G6, F.Cu at (150.5, 110.5)
- added Q9: Q_NMOS, footprints:QNM30N20AJ-PDFN-8L_L3.3-W3.3-P0.65-BL_XINFEIHONG_FH1404G6, F.Cu at (139.0, 106.0)
- added R1: 10m, Resistor_SMD:R_1206_3216Metric, F.Cu at (148.8, 97.7)
- added R10: 160k, Resistor_SMD:R_0603_1608Metric, F.Cu at (82.7, 88.0)
- added R11: 220k, Resistor_SMD:R_0402_1005Metric, F.Cu at (90.9, 85.7)
- added R12: 0, Resistor_SMD:R_0603_1608Metric, F.Cu at (82.7, 90.5)
- added R13: 220k, Resistor_SMD:R_0402_1005Metric, F.Cu at (90.9, 87.6)
- added R14: 40.2k, Resistor_SMD:R_0603_1608Metric, F.Cu at (86.7, 82.9)
- added R15: 10k, Resistor_SMD:R_0805_2012Metric, F.Cu at (86.5, 89.4)
- added R16: 10k, Resistor_SMD:R_0805_2012Metric, F.Cu at (64.4, 115.7)
- added R17: 10, Resistor_SMD:R_0402_1005Metric, F.Cu at (48.2, 151.5)
- added R18: 10k, Resistor_SMD:R_0805_2012Metric, F.Cu at (64.4, 118.7)
- added R19: 10k, Resistor_SMD:R_0805_2012Metric, F.Cu at (64.4, 121.6)
- added R2: 10m, Resistor_SMD:R_1206_3216Metric, F.Cu at (148.8, 101.0)
- added R20: 390k, Resistor_SMD:R_0603_1608Metric, F.Cu at (42.6, 144.8)
- added R21: 220k, Resistor_SMD:R_0402_1005Metric, F.Cu at (48.2, 153.4)
- added R22: 137k, Resistor_SMD:R_0603_1608Metric, F.Cu at (42.6, 147.3)
- added R23: 220k, Resistor_SMD:R_0402_1005Metric, F.Cu at (48.2, 155.4)
- added R24: 40.2k, Resistor_SMD:R_0603_1608Metric, F.Cu at (42.6, 149.8)
- added R25: 10k, Resistor_SMD:R_0805_2012Metric, F.Cu at (68.8, 109.8)
- added R26: 10k, Resistor_SMD:R_0805_2012Metric, F.Cu at (68.8, 112.8)
- added R27: 300, Resistor_SMD:R_1206_3216Metric, F.Cu at (149.5, 123.0)
- added R28: 10M, Resistor_SMD:R_0402_1005Metric, F.Cu at (147.7, 127.5)
- added R29: 10M, Resistor_SMD:R_0402_1005Metric, F.Cu at (143.7, 122.0)
- added R3: 4.7, Resistor_SMD:R_0603_1608Metric, F.Cu at (38.6, 147.3)
- added R30: 10k, Resistor_SMD:R_0805_2012Metric, F.Cu at (68.8, 115.7)
- added R31: 10k, Resistor_SMD:R_0805_2012Metric, F.Cu at (68.8, 118.7)
- added R32: 10M, Resistor_SMD:R_0402_1005Metric, F.Cu at (143.7, 124.0)
- added R33: 5.1k, Resistor_SMD:R_0402_1005Metric, F.Cu at (143.7, 126.0)
- added R34: 5.1k, Resistor_SMD:R_0402_1005Metric, F.Cu at (143.7, 128.0)
- added R35: 100, Resistor_SMD:R_0402_1005Metric, F.Cu at (143.7, 130.0)
- added R36: 5.1k, Resistor_SMD:R_0402_1005Metric, F.Cu at (143.7, 131.9)
- added R37: 2.2, Resistor_SMD:R_0805_2012Metric, F.Cu at (68.8, 121.6)
- added R38: 2.2, Resistor_SMD:R_0805_2012Metric, F.Cu at (73.2, 109.8)
- added R39: 2.2, Resistor_SMD:R_0805_2012Metric, F.Cu at (73.2, 112.8)
- added R4: 4.7, Resistor_SMD:R_0603_1608Metric, F.Cu at (38.6, 149.8)
- added R40: 2.2, Resistor_SMD:R_0805_2012Metric, F.Cu at (73.2, 115.7)
- added R41: 100, Resistor_SMD:R_0402_1005Metric, F.Cu at (51.1, 153.4)
- added R42: 4.7k, Resistor_SMD:R_0402_1005Metric, F.Cu at (51.1, 155.4)
- added R43: 4.7k, Resistor_SMD:R_0402_1005Metric, F.Cu at (51.1, 157.4)
- added R44: 4.7k, Resistor_SMD:R_0402_1005Metric, F.Cu at (54.0, 141.5)
- added R45: 100, Resistor_SMD:R_0402_1005Metric, F.Cu at (54.0, 143.5)
- added R46: 0, Resistor_SMD:R_0603_1608Metric, F.Cu at (42.6, 152.3)
- added R47: 100, Resistor_SMD:R_0402_1005Metric, F.Cu at (54.0, 145.5)
- added R48: 10, Resistor_SMD:R_0402_1005Metric, F.Cu at (54.0, 147.5)
- added R49: 100, Resistor_SMD:R_0402_1005Metric, F.Cu at (54.0, 149.5)
- added R5: 1, Resistor_SMD:R_0402_1005Metric, F.Cu at (48.2, 141.5)
- added R50: 10m, Resistor_SMD:R_1206_3216Metric, F.Cu at (115.0, 137.0)
- added R51: 100, Resistor_SMD:R_0402_1005Metric, F.Cu at (138.0, 115.2)
- added R52: 100, Resistor_SMD:R_0402_1005Metric, F.Cu at (140.3, 115.2)
- added R53: 1m, Resistor_SMD:R_1206_3216Metric, F.Cu at (140.8, 112.0)
- added R54: 200, Resistor_SMD:R_0402_1005Metric_Pad0.72x0.64mm_HandSolder, F.Cu at (78.4, 105.2)
- added R55: 100, Resistor_SMD:R_0402_1005Metric, F.Cu at (54.0, 155.4)
- added R56: 1k, Resistor_SMD:R_0603_1608Metric, F.Cu at (42.6, 154.8)
- added R57: 5.6k, Resistor_SMD:R_0402_1005Metric, F.Cu at (54.0, 157.4)
- added R58: 4.7k, Resistor_SMD:R_0402_1005Metric, F.Cu at (56.9, 141.5)
- added R59: 4.7k, Resistor_SMD:R_0402_1005Metric, F.Cu at (56.9, 143.5)
- added R6: 10, Resistor_SMD:R_0402_1005Metric, F.Cu at (48.2, 143.5)
- added R60: 220k, Resistor_SMD:R_0402_1005Metric, F.Cu at (121.0, 136.8)
- added R61: 10, Resistor_SMD:R_0402_1005Metric, F.Cu at (56.9, 147.5)
- added R62: 4.7k, Resistor_SMD:R_0402_1005Metric, F.Cu at (56.9, 149.5)
- added R63: 200, Resistor_SMD:R_0402_1005Metric_Pad0.72x0.64mm_HandSolder, F.Cu at (78.4, 107.2)
- added R64: 100, Resistor_SMD:R_0402_1005Metric, F.Cu at (56.9, 151.5)
- added R65: 22k, Resistor_SMD:R_0402_1005Metric, F.Cu at (121.0, 139.5)
- added R7: 10, Resistor_SMD:R_0402_1005Metric, F.Cu at (48.2, 145.5)
- added R8: DNP, Resistor_SMD:R_0603_1608Metric, F.Cu at (82.7, 85.5)
- added R9: 10k, Resistor_SMD:R_0805_2012Metric, F.Cu at (86.5, 86.4)
- added SW1: SW_Push, Button_Switch_THT:SW_PUSH_6mm, F.Cu at (154.2, 85.2)
- added SW2: SW_Push, Connector_Wire:SolderWire-0.127sqmm_1x02_P3.7mm_D0.48mm_OD1mm, F.Cu at (172.2, 106.2)
- added SW3: SW_Push, Button_Switch_THT:SW_PUSH_6mm, F.Cu at (96.8, 118.2)
- added TH1: 10k, Connector_Wire:SolderWire-0.127sqmm_1x02_P3.7mm_D0.48mm_OD1mm, F.Cu at (172.2, 110.0)
- added U1: TPS25730DREFR, footprints:REF0038A-MFG, F.Cu at (112.9, 95.1)
- added U2: BQ25713RSNR, footprints:RSN32_TEX, F.Cu at (123.8, 111.0)
- added U3: TPS25762DQRQLRQ1, footprints:RQL0029A-MFG, F.Cu at (116.5, 131.7)
- added U4: nRF54L10-QFXX, Package_DFN_QFN:QFN-48-1EP_6x6mm_P0.4mm_EP4.6x4.6mm_ThermalVias, F.Cu at (156.0, 118.0)
- added U5: BQ4050RSMR, footprints:VQFN-32_L4.0-W4.0-P0.40-TL-EP1.4, F.Cu at (142.1, 100.3)
- added U6: AT24C256C-SSHL-T, footprints:SOIC-8_L4.9-W3.9-P1.27-LS6.0-BL, F.Cu at (123.1, 130.1)
- added X1: 32MHz, footprints:CRYSTAL-SMD_4P-L2.0-W1.6-BL-A, F.Cu at (156.5, 105.0)

Commit message: mv
Parts:
- moved R3 171.0 mm to (208.4, 127.2)
- moved R4 171.0 mm to (208.4, 129.8)
- moved R24 168.7 mm to (210.9, 139.8)
- moved C39 161.3 mm to (212.3, 141.8)
- moved C41 160.6 mm to (213.8, 139.5)
- moved C22 156.7 mm to (204.7, 125.6)
- moved C23 156.7 mm to (204.7, 127.6)
- moved C40 150.6 mm to (201.6, 140.2)
- moved R26 131.6 mm to (197.5, 140.5)
- moved R16 119.8 mm to (184.2, 112.5)
- moved R18 119.8 mm to (184.2, 115.5)
- moved C10 113.8 mm to (167.4, 93.9)
- moved C8 113.8 mm to (167.4, 87.8)
- moved C9 113.8 mm to (167.4, 90.8)
- moved C4 112.4 mm to (171.8, 86.0)
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Connections:
- C34 pad 1: INPUT_VBUS -> (no net)
- C34 pad 2: GND -> (no net)
- C40 pad 1: GND -> (no net)
- C40 pad 2: Net-(U2-COMP2) -> (no net)
- C42 pad 1: Net-(C42-Pad1) -> (no net)
- C42 pad 2: GND -> (no net)
- R1 pad 1: INPUT_PWR -> (no net)
- R1 pad 2: Net-(C22-Pad1) -> (no net)
- R25 pad 1: 4P -> (no net)
- R25 pad 2: Net-(R25-Pad2) -> (no net)
Other:
- board text added: "TPS25762-Q1 TVSP"
- board text added: "acp acn current sensing"
- board text added: "bq25713 comp1"
- board text added: "bq25713 comp2"
- board text added: "bq25713 in"
- board text added: "bq25713 vbus"
- board text added: "bq25713 vsys caps"
- board text added: "tps25730 adcin"
- board text added: "tps25762-q1 switching"

Commit message: firmware init
Parts:
- moved Q3 11.8 mm to (106.2, 112.0)
- moved Q4 10.7 mm to (102.1, 106.7)
- moved Q5 10.7 mm to (106.6, 106.7)
- moved U2 2.63 mm to (125.1, 113.3)
- moved Q1 2.33 mm to (97.4, 102.7)
- moved Q2 2.33 mm to (92.8, 102.9)
- moved C12 2.25 mm to (101.2, 91.3)
- moved C2 2.25 mm to (98.0, 91.0)
- moved C27 2.25 mm to (98.0, 93.0)
- moved C28 2.25 mm to (98.0, 95.2)
- moved C3 2.25 mm to (98.0, 97.3)
- moved C68 2.25 mm to (94.8, 123.0)
- moved C69 2.25 mm to (99.5, 133.2)
- moved C70 2.25 mm to (99.5, 135.2)
- moved D10 2.25 mm to (92.3, 115.2)
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Other:
- board size 74 x 51.5 mm -> 74 x 56 mm
- board text added: "SW1"
Changed lines of the file:
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@@
 	(footprint "LED_SMD:LED_0603_1608Metric"
 		(layer "F.Cu")
-		(at 92.2875 117.41)
+		(at 92.2875 115.16)
 		(descr "LED SMD 0603 (1608 Metric), square (rectangular) end terminal, IPC-7351 nominal, (Body size source: http://www.tortai-tech.com/upload/download/2011102023233369053.pdf)")
 		(tags "LED")
@@
 	(footprint "Capacitor_SMD:C_0402_1005Metric"
 		(layer "F.Cu")
-		(at 98 95.27 90)
+		(at 98 93.02 90)
 		(descr "Capacitor SMD 0402 (1005 Metric), square (rectangular) end terminal, IPC-7351 nominal, (Body size source: IPC-SM-782 page 76, https://www.pcb-3d.com/wordpress/wp-content/uploads/ipc-sm-782a_amendment_1_and_2.pdf)")
 		(tags "capacitor")
@@
 	(footprint "footprints:QNM30N20AJ-PDFN-8L_L3.3-W3.3-P0.65-BL_XINFEIHONG_FH1404G6"
 		(layer "F.Cu")
-		(at 93.81 104.97)
+		(at 92.75 102.89)
 		(property "Reference" "Q2"
 			(at 0 -2.55 0)
@@
 	(footprint "Capacitor_SMD:C_0402_1005Metric"
 		(layer "F.Cu")
-		(at 98 97.5 90)
+		(at 98 95.25 90)
 		(descr "Capacitor SMD 0402 (1005 Metric), square (rectangular) end terminal, IPC-7351 nominal, (Body size source: IPC-SM-782 page 76, https://www.pcb-3d.com/wordpress/wp-content/uploads/ipc-sm-782a_amendment_1_and_2.pdf)")
 		(tags "capacitor")
@@
 			(at 3.25 -2 0)
 			(layer "User.1")
+			(hide yes)
 			(effects
 				(font
@@
 	(footprint "footprints:CAP-SMD_L7.3-W6.1_TCN4227M025R0100"
 		(layer "F.Cu")
-		(at 94.75 125.25 180)
+		(at 94.75 123 180)
 		(property "Reference" "C68"
 			(at 0 -4 0)
@@
 	(footprint "footprints:ZC015P2G-POWERTDFN-8_L3.1-W3.1-P0.65-LS3.3-BL"
 		(layer "F.Cu")
-		(at 116.81 117.29)
+		(at 106.25 112.03)
 		(property "Reference" "Q3"
 			(at 0 -2.5 0)
@@
 	(footprint "Capacitor_SMD:C_0805_2012Metric"
 		(layer "F.Cu")
-		(at 101.25 93.55 90)
+		(at 101.25 91.3 90)
 		(descr "Capacitor SMD 0805 (2012 Metric), square (rectangular) end terminal, IPC-7351 nominal, (Body size source: IPC-SM-782 page 76, https://www.pcb-3d.com/wordpress/wp-content/uploads/ipc-sm-782a_amendment_1_and_2.pdf, https://docs.google.com/spreadsheets/d/1BsfQQcO9C6DZCsRaXUlFlo91Tg2WpOkGARC1WS5S8t0/edit?usp=sharing)")
 		(tags "capacitor")
@@
 	(footprint "Capacitor_SMD:C_0402_1005Metric"
 		(layer "F.Cu")
-		(at 99.5 135.5)
+		(at 99.5 133.25)
 		(descr "Capacitor SMD 0402 (1005 Metric), square (rectangular) end terminal, IPC-7351 nominal, (Body size source: IPC-SM-782 page 76, https://www.pcb-3d.com/wordpress/wp-content/uploads/ipc-sm-782a_amendment_1_and_2.pdf)")
 		(tags "capacitor")
@@
 	(footprint "LED_SMD:LED_0603_1608Metric"
 		(layer "F.Cu")
-		(at 92.2875 112.41)
+		(at 92.2875 110.16)
 		(descr "LED SMD 0603 (1608 Metric), square (rectangular) end terminal, IPC-7351 nominal, (Body size source: http://www.tortai-tech.com/upload/download/2011102023233369053.pdf)")
 		(tags "LED")
@@
 	(footprint "footprints:QNM30N20AJ-PDFN-8L_L3.3-W3.3-P0.65-BL_XINFEIHONG_FH1404G6"
 		(layer "F.Cu")
-		(at 108.25 115.5)
+		(at 102.06 106.72)
 		(property "Reference" "Q4"
-			(at 0 -2.55 0)
+			(at 0 -4.8 0)
 			(layer "User.1")
 			(effects
@@
 		)
 		(property "Value" "Q_NMOS"
-			(at 0.02 2.49 0)
+			(at 0.02 0.24 0)
 			(layer "F.Fab")
 			(effects
@@
 		)
 		(fp_text user "${REFERENCE}"
-			(at 0 0 0)
+			(at 0 -2.25 0)
 			(layer "F.Fab")
 			(effects
@@
 	(footprint "footprints:QNM30N20AJ-PDFN-8L_L3.3-W3.3-P0.65-BL_XINFEIHONG_FH1404G6"
 		(layer "F.Cu")
-		(at 112.75 115.5)
+		(at 106.56 106.72)
 		(property "Reference" "Q5"
 			(at 0 -2.55 0)
@@
 	(footprint "Capacitor_SMD:C_0402_1005Metric"
 		(layer "F.Cu")
-		(at 98 99.54 -90)
+		(at 98 97.29 -90)
 		(descr "Capacitor SMD 0402 (1005 Metric), square (rectangular) end terminal, IPC-7351 nominal, (Body size source: IPC-SM-782 page 76, https://www.pcb-3d.com/wordpress/wp-content/uploads/ipc-sm-782a_amendment_1_and_2.pdf)")
 		(tags "capacitor")
@@
 	(footprint "footprints:USB-C-SMD_TYPE-C16PIN"
 		(layer "F.Cu")
-		(at 94.25 133.75 -90)
+		(at 94.25 131.5 -90)
 		(property "Reference" "J2"
 			(at 0 -3.284701 90)
@@
 	(footprint "footprints:QNM30N20AJ-PDFN-8L_L3.3-W3.3-P0.65-BL_XINFEIHONG_FH1404G6"
 		(layer "F.Cu")
-		(at 98.5 104.75)
+		(at 97.44 102.67)
 		(property "Reference" "Q1"
 			(at 0 -2.55 0)
@@
 	(footprint "Capacitor_SMD:C_0402_1005Metric"
 		(layer "F.Cu")
-		(at 99.5 137.47)
+		(at 99.5 135.22)
 		(descr "Capacitor SMD 0402 (1005 Metric), square (rectangular) end terminal, IPC-7351 nominal, (Body size source: IPC-SM-782 page 76, https://www.pcb-3d.com/wordpress/wp-content/uploads/ipc-sm-782a_amendment_1_and_2.pdf)")
 		(tags "capacitor")
@@
 	(footprint "Button_Switch_THT:SW_PUSH_6mm"
 		(layer "F.Cu")
-		(at 96.75 118.25 90)
+		(at 96.5 117.5 90)
 		(descr "Generic 6mm SW tactile push button")
 		(tags "tact sw push 6mm")
@@
 	(footprint "footprints:USB-C-SMD_TYPE-C16PIN"
 		(layer "F.Cu")
-		(at 94.095 96.5 -90)
+		(at 94.095 94.25 -90)
 		(property "Reference" "J1"
 			(at -0.02 -4.224701 90)
@@
 	(footprint "footprints:RSN32_TEX"
 		(layer "F.Cu")
-		(at 123.7585 110.999999)
+		(at 125.1 113.2585)
 		(tags "BQ25713BRSNR ")
 		(property "Reference" "U2"
@@
 	(footprint "LED_SMD:LED_0603_1608Metric"
 		(layer "F.Cu")
-		(at 92.2875 120)
+		(at 92.2875 117.75)
 		(descr "LED SMD 0603 (1608 Metric), square (rectangular) end terminal, IPC-7351 nominal, (Body size source: http://www.tortai-tech.com/upload/download/2011102023233369053.pdf)")
 		(tags "LED")
@@
 	(footprint "LED_SMD:LED_0603_1608Metric"
 		(layer "F.Cu")
-		(at 92.2875 110)
+		(at 92.2875 107.75)
 		(descr "LED SMD 0603 (1608 Metric), square (rectangular) end terminal, IPC-7351 nominal, (Body size source: http://www.tortai-tech.com/upload/download/2011102023233369053.pdf)")
 		(tags "LED")
@@
 	(footprint "Capacitor_SMD:C_0402_1005Metric"
 		(layer "F.Cu")
-		(at 98 93.27 90)
+		(at 98 91.02 90)
 		(descr "Capacitor SMD 0402 (1005 Metric), square (rectangular) end terminal, IPC-7351 nominal, (Body size source: IPC-SM-782 page 76, https://www.pcb-3d.com/wordpress/wp-content/uploads/ipc-sm-782a_amendment_1_and_2.pdf)")
 		(tags "capacitor")
@@
 	(footprint "LED_SMD:LED_0603_1608Metric"
 		(layer "F.Cu")
-		(at 92.2875 115)
+		(at 92.2875 112.75)
 		(descr "LED SMD 0603 (1608 Metric), square (rectangular) end terminal, IPC-7351 nominal, (Body size source: http://www.tortai-tech.com/upload/download/2011102023233369053.pdf)")
 		(tags "LED")
@@
 	)
 	(gr_rect
-		(start 88.75 17)
-		(end 107.25 82)
+		(start 192.5 19.5)
+		(end 211 84.5)
 		(stroke
 			(width 0.1)
@@
 	)
 	(gr_rect
-		(start 107.5 17)
-		(end 126 82)
+		(start 211.25 19.5)
+		(end 229.75 84.5)
 		(stroke
 			(width 0.1)
@@
 	)
 	(gr_rect
-		(start 126.25 17)
-		(end 144.75 82)
+		(start 230 19.5)
+		(end 248.5 84.5)
 		(stroke
 			(width 0.1)
@@
 	)
 	(gr_rect
-		(start 145 17)
-		(end 163.5 82)
+		(start 248.75 19.5)
+		(end 267.25 84.5)
 		(stroke
 			(width 0.1)
@@
 	)
 	(gr_rect
-		(start 89 89.5)
+		(start 89 85)
 		(end 163 141)
 		(stroke
@@
 	)
 	(gr_text "18650"
-		(at 90.75 81 0)
+		(at 194.5 83.5 0)
 		(layer "Dwgs.User")
 		(effects
@@
 	)
 	(gr_text "18650"
-		(at 109.5 81 0)
+		(at 213.25 83.5 0)
 		(layer "Dwgs.User")
 		(effects
@@
 	)
 	(gr_text "18650"
-		(at 128.25 81 0)
+		(at 232 83.5 0)
 		(layer "Dwgs.User")
 		(effects
@@
 	)
 	(gr_text "18650"
-		(at 147 81 0)
+		(at 250.75 83.5 0)
 		(layer "Dwgs.User")
 		(effects
@@
 		)
 	)
+	(gr_text "SW1"
+		(at 157.75 83.5 0)
+		(layer "User.1")
+		(effects
+			(font
+				(size 0.25 0.25)
+				(thickness 0.1)
+			)
+		)
+	)
 	(gr_text "tps25730 adcin"
-		(at 76.5 81 0)
+		(at 81.75 79.25 0)
 		(layer "User.1")
 		(effects
