File: pcb/FindMyCharger.kicad_pcb (KiCad board)
At the start: 4 copper layers, 74 x 56 mm, 211 parts, among them J1 USB_C_Receptacle_USB2.0_16P, J2 USB_C_Receptacle_USB2.0_16P, J3 Battery_Connector, Q1 Q_NMOS, Q2 Q_NMOS, Q3 Q_PMOS, Q4 Q_NMOS, Q5 Q_NMOS, Q6 Q_PMOS, Q7 Q_NMOS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

Commit message: a
Parts:
- removed R12: 0, Resistor_SMD:R_0603_1608Metric
- removed R8: DNP, Resistor_SMD:R_0603_1608Metric
- moved R4 110.9 mm to (100.4, 104.5)
- moved R3 110.1 mm to (100.4, 106.0)
- moved R1 106.4 mm to (103.8, 104.5), turned to -90 degrees
- moved C32 101.8 mm to (104.0, 108.5), turned to -90 degrees
- moved H1 100.9 mm to (91.2, 87.0)
- moved C23 98.8 mm to (107.8, 108.8)
- moved C22 98.6 mm to (107.8, 107.8)
- moved C31 97.3 mm to (105.5, 108.5), turned to -90 degrees
- moved H2 82.7 mm to (94.8, 87.0)
- moved C34 73.5 mm to (100.5, 103.0)
- moved R5 73.0 mm to (100.0, 101.5)
- moved C21 67.8 mm to (108.8, 94.7), turned to 90 degrees
- moved C20 66.6 mm to (106.8, 94.7), turned to 90 degrees
- moved C19 65.5 mm to (104.8, 94.7), turned to 90 degrees
- moved C18 62.1 mm to (108.8, 98.2), turned to 90 degrees
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Connections:
- C15 pad 1: (no net) -> INPUT_PWR
- C15 pad 2: (no net) -> GND
- C29 pad 2: GND -> PD_ADCIN1
- C34 pad 1: (no net) -> INPUT_VBUS
- C34 pad 2: (no net) -> GND
- C35 pad 2: GND -> PD_ADCIN1
- C36 pad 2: GND -> PD_ADCIN1
- C50 pad 2: GND -> PD_ADCIN1
- C51 pad 2: GND -> PD_ADCIN1
- C54 pad 2: GND -> PD_ADCIN1
- C59 pad 2: GND -> PD_ADCIN1
- C60 pad 2: GND -> PD_ADCIN1
- C61 pad 2: GND -> PD_ADCIN1
- C75 pad 2: GND -> PD_ADCIN1
- C76 pad 2: GND -> PD_ADCIN1
- C77 pad 2: GND -> PD_ADCIN1
- C81 pad 2: GND -> PD_ADCIN1
- C85 pad 2: GND -> PD_ADCIN1
- R1 pad 1: (no net) -> INPUT_PWR
- R1 pad 2: (no net) -> Net-(C22-Pad1)
- R21 pad 2: GND -> PD_ADCIN1
- R22 pad 2: GND -> PD_ADCIN1
- R23 pad 2: GND -> PD_ADCIN1
- R31 pad 2: GND -> PD_ADCIN1
- R61 pad 2: GND -> PD_ADCIN1
- R62 pad 2: GND -> PD_ADCIN1
- U1 pad 2: PD_ADCIN1 -> GND

Commit message: a
Parts:
- removed H3: iCHG, TestPoint:TestPoint_Pad_D2.5mm
- moved C41 99.8 mm to (118.2, 110.5), turned to 90 degrees
- moved C39 97.8 mm to (119.2, 111.6), turned to 90 degrees
- moved R24 96.7 mm to (118.0, 113.1), turned to 90 degrees
- moved C42 91.7 mm to (114.2, 113.8)
- moved C40 90.3 mm to (115.8, 112.2)
- moved R26 89.4 mm to (112.9, 111.8)
- moved C54 76.8 mm to (145.8, 105.8)
- moved C59 76.8 mm to (145.8, 108.8)
- moved C61 76.8 mm to (145.8, 111.8)
- moved D5 72.5 mm to (99.0, 135.9), turned to 180 degrees
- moved R22 67.2 mm to (131.7, 110.8)
- moved R20 63.8 mm to (128.5, 110.2), turned to 90 degrees
- moved C36 63.7 mm to (131.5, 109.5)
- moved R23 59.6 mm to (128.2, 113.0), turned to 90 degrees
- moved C26 59.5 mm to (120.5, 92.8), turned to 90 degrees
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Connections:
- C12 pad 1: (no net) -> VBUS_IN
- C12 pad 2: (no net) -> GND
- C35 pad 1: INPUT_VDDA -> (no net)
- C35 pad 2: PD_ADCIN1 -> (no net)
- C36 pad 1: INPUT_IADPT -> (no net)
- C36 pad 2: PD_ADCIN1 -> (no net)
- C52 pad 1: BMS_VC3 -> BMS_VC4
- C52 pad 2: BMS_VC4 -> Net-(J3-PadBAT3)
- C53 pad 1: BMS_VC2 -> (no net)
- C53 pad 2: BMS_VC3 -> (no net)
- C56 pad 1: BMS_VC1 -> (no net)
- C56 pad 2: BMS_VC2 -> (no net)
- C57 pad 1: CHGND -> Net-(J3-PadBAT1)
- C57 pad 2: BMS_VC1 -> CHGND
- C68 pad 1: (no net) -> VBUS_OUT
- C68 pad 2: (no net) -> GND
- R17 pad 1: INPUT_REGN -> (no net)
- R17 pad 2: INPUT_VDDA -> (no net)
- R20 pad 1: INPUT_VDDA -> (no net)
- R20 pad 2: INPUT_ILIM_HIZ -> (no net)
- R21 pad 1: INPUT_CELL_BATPRESZ -> (no net)
- R21 pad 2: PD_ADCIN1 -> (no net)
- R22 pad 1: INPUT_IADPT -> (no net)
- R22 pad 2: PD_ADCIN1 -> (no net)
- R23 pad 1: INPUT_ILIM_HIZ -> (no net)
- R23 pad 2: PD_ADCIN1 -> (no net)
- R27 pad 2: Net-(Q6-PadD) -> (no net)
- R29 pad 1: 4P -> (no net)
- R29 pad 2: Net-(Q7-PadG) -> (no net)
Routing:
- net DP_OUT: track 0.00 -> 12.5 mm
- net CC1_OUT: track 0.00 -> 7.50 mm
- net VBUS_IN: track 0.00 -> 5.85 mm
- net CC2_OUT: track 0.00 -> 4.95 mm
- net DM_OUT: track 0.00 -> 2.69 mm
- net CC2_IN: track 0.00 -> 1.56 mm
- net CC1_IN: track 0.00 -> 1.55 mm
- net GND: track 0.00 -> 0.99 mm
Other:
- board text removed: "TPS25762-Q1 TVSP"
- board text removed: "bq25713 comp1"
- board text removed: "bq25713 comp2"
- board text removed: "bq25713 in"
- board text removed: "bq25713 vbus"
- board text removed: "tps25730 adcin"
- board text removed: "tps25762-q1 switching"

Commit message: route
Parts:
- removed C71, C72: 0.1uF, Capacitor_SMD:C_0402_1005Metric
- moved R56 98.2 mm to (156.4, 112.5)
- moved H14 79.2 mm to (100.5, 128.0)
- moved R16 73.0 mm to (113.0, 96.2), turned to 90 degrees
- moved R18 71.5 mm to (115.2, 96.3), turned to 90 degrees
- moved H5 70.3 mm to (123.0, 119.8)
- moved H12 67.0 mm to (119.0, 101.5), turned to 90 degrees
- moved R46 63.4 mm to (127.2, 130.2)
- moved H8 61.4 mm to (118.8, 105.2), turned to 90 degrees
- moved H10 60.1 mm to (118.5, 108.8)
- moved D4 59.3 mm to (110.5, 125.6)
- moved R48 58.7 mm to (136.0, 133.5)
- moved H4 57.4 mm to (111.2, 121.0)
- moved H15 54.2 mm to (127.8, 118.0)
- moved H6 53.0 mm to (118.3, 120.2)
- moved R43 48.2 mm to (114.5, 127.8)
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Connections:
- C1 pad 1: (no net) -> Net-(U1-VIN_3V3)
- C1 pad 2: (no net) -> GND
- C55 pad 1: (no net) -> OUTPUT_CSN_BUS
- C55 pad 2: (no net) -> OUTPUT_CSP
- D1 pad 1: (no net) -> GND
- D1 pad 3: (no net) -> VBUS_IN
- H9 pad 1: Net-(H9-Pad1) -> (no net)
- L3 pad 1: (no net) -> Net-(U4-DCC)
- L3 pad 2: (no net) -> Net-(U4-DECD)
- R50 pad 1: (no net) -> OUTPUT_OUT
- R50 pad 2: (no net) -> VBUS_OUT
- X1 pad 1: (no net) -> Net-(U4-XC1)
- X1 pad 2: (no net) -> GND
- X1 pad 3: (no net) -> Net-(U4-XC2)
- X1 pad 4: (no net) -> GND
Routing:
- net GND: track 0.99 -> 110.3 mm, vias 0 -> 14
- net VBUS_OUT: track 0.00 -> 78.9 mm, vias 0 -> 2
- net OUTPUT_LDO_3V3: track 0.00 -> 58.6 mm, vias 0 -> 6
- net BMS_SRN: track 0.00 -> 27.5 mm
- net INPUT_PWR: track 0.00 -> 25.6 mm
- net INPUT_VSYS: track 0.00 -> 25.2 mm
- net OUTPUT_SW2: track 0.00 -> 22.5 mm
- net Net-(U3-GPIO1_IRQ2(o)): track 0.00 -> 21.1 mm
- net CHG_SDA: track 0.00 -> 19.1 mm
- net OUTPUT_OUT: track 0.00 -> 18.9 mm
- net PD_ADCIN4: track 0.00 -> 18.8 mm, vias 0 -> 2
- net CHG_SCL: track 0.00 -> 17.3 mm
- net Net-(U3-GPIO2_I2C_SCL2): track 0.00 -> 15.8 mm, vias 0 -> 2
- net OUTPUT_SW1: track 0.00 -> 15.6 mm
- net BMS_VC1: track 0.00 -> 14.9 mm
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- added copper zone on In1.Cu, net GND

Commit message: cleanup
Connections:
- FB1 pad 1: (no net) -> Net-(U4-DECD)
- FB1 pad 2: (no net) -> Net-(U4-DECA)
Routing:
- net OUTPUT_LDO_3V3: track 58.6 -> 175.3 mm, vias 6 -> 9
- net 4P: track 0.00 -> 65.0 mm, vias 0 -> 1
- net GND: track 110.3 -> 175.0 mm, vias 14 -> 28
- net VBUS_OUT: track 78.9 -> 138.4 mm
- net CHG_SCL: track 17.3 -> 59.8 mm, vias 0 -> 1
- net Net-(Q6-PadS): track 0.00 -> 41.4 mm
- net OUTPUT_BOOT1: track 0.00 -> 35.9 mm, vias 0 -> 2
- net Net-(U4-DECA): track 0.00 -> 35.9 mm
- net OUTPUT_OUT: track 18.9 -> 50.0 mm, vias 0 -> 2
- net Net-(U4-DCC): track 0.00 -> 24.1 mm
- net PD_ADCIN1: track 9.91 -> 34.0 mm, vias 0 -> 2
- net Net-(AE1-A): track 0.00 -> 21.9 mm, vias 0 -> 2
- net Net-(H8-Pad1): track 0.00 -> 20.8 mm, vias 0 -> 1
- net Net-(C76-Pad1): track 0.00 -> 20.7 mm
- net Net-(U4-DECD): track 0.00 -> 19.9 mm, vias 0 -> 2
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